File: KICAD/MP3_Player/MP3_Player.kicad_sch (KiCad schematic)
At the start: 0 parts

Commit message: Add files via upload
Other:
- sheet Audio ports: added DAC_BCK, DAC_DIN, DAC_LRCK, DAC_XSMT; removed CODEC_BCK, CODEC_DIN, CODEC_LRCK, CODEC_XSMT
- sheet MCU ports: added DAC_BCK, DAC_DIN, DAC_LRCK, DAC_XSMT; removed CODEC_BCK, CODEC_DIN, CODEC_LRCK, CODEC_XSMT
Changed lines of the file:
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@@
+	(wire
+		(pts
+			(xy 166.37 39.37) (xy 218.44 39.37)
+		)
+		(stroke
+			(width 0)
+			(type default)
+		)
+	)
 	(wire
 		(pts
@@
 		(pts
 			(xy 33.02 44.45) (xy 33.02 168.91)
-		)
-		(stroke
-			(width 0)
-			(type default)
-		)
-	)
-	(wire
-		(pts
-			(xy 166.37 39.37) (xy 218.44 39.37)
 		)
 		(stroke
@@
 			)
 		)
-		(pin "CODEC_BCK" input
-			(at 218.44 36.83 180)
-			(effects
-				(font
-					(size 1.27 1.27)
-				)
-				(justify left)
-			)
-		)
 		(pin "MIC_WS" input
 			(at 218.44 54.61 180)
@@
 			)
 		)
-		(pin "CODEC_LRCK" input
-			(at 218.44 39.37 180)
-			(effects
-				(font
-					(size 1.27 1.27)
-				)
-				(justify left)
-			)
-		)
-		(pin "CODEC_DIN" input
-			(at 218.44 41.91 180)
-			(effects
-				(font
-					(size 1.27 1.27)
-				)
-				(justify left)
-			)
-		)
-		(pin "CODEC_XSMT" input
-			(at 218.44 44.45 180)
-			(effects
-				(font
-					(size 1.27 1.27)
-				)
-				(justify left)
-			)
-		)
 		(pin "MIC_SCK" input
 			(at 218.44 49.53 180)
+			(effects
+				(font
+					(size 1.27 1.27)
+				)
+				(justify left)
+			)
+		)
+		(pin "DAC_DIN" input
+			(at 218.44 41.91 180)
+			(effects
+				(font
+					(size 1.27 1.27)
+				)
+				(justify left)
+			)
+		)
+		(pin "DAC_XSMT" input
+			(at 218.44 44.45 180)
+			(effects
+				(font
+					(size 1.27 1.27)
+				)
+				(justify left)
+			)
+		)
+		(pin "DAC_LRCK" input
+			(at 218.44 39.37 180)
+			(effects
+				(font
+					(size 1.27 1.27)
+				)
+				(justify left)
+			)
+		)
+		(pin "DAC_BCK" input
+			(at 218.44 36.83 180)
 			(effects
 				(font
@@
 	(sheet
 		(at 137.16 31.75)
-		(size 29.21 101.6)
+		(size 29.21 106.68)
 		(exclude_from_sim no)
 		(in_bom yes)
@@
 			)
 		)
-		(pin "CODEC_BCK" output
-			(at 166.37 36.83 0)
-			(effects
-				(font
-					(size 1.27 1.27)
-				)
-				(justify right)
-			)
-		)
-		(pin "CODEC_DIN" output
-			(at 166.37 41.91 0)
-			(effects
-				(font
-					(size 1.27 1.27)
-				)
-				(justify right)
-			)
-		)
-		(pin "CODEC_LRCK" output
-			(at 166.37 39.37 0)
-			(effects
-				(font
-					(size 1.27 1.27)
-				)
-				(justify right)
-			)
-		)
-		(pin "CODEC_XSMT" output
-			(at 166.37 44.45 0)
-			(effects
-				(font
-					(size 1.27 1.27)
-				)
-				(justify right)
-			)
-		)
 		(pin "MIC_SCK" output
 			(at 166.37 49.53 0)
@@
 			(effects
 				(font
+					(size 1.27 1.27)
+				)
+				(justify right)
+			)
+		)
+		(pin "DAC_BCK" output
+			(at 166.37 36.83 0)
+			(effects
+				(font
+					(size 1.27 1.27)
+				)
+				(justify right)
+			)
+		)
+		(pin "DAC_DIN" output
+			(at 166.37 41.91 0)
+			(effects
+				(font
+					(size 1.27 1.27)
+				)
+				(justify right)
+			)
+		)
+		(pin "DAC_LRCK" output
+			(at 166.37 39.37 0)
+			(effects
+				(font
+					(size 1.27 1.27)
+				)
+				(justify right)
+			)
+		)
+		(pin "DAC_XSMT" output
+			(at 166.37 44.45 0)
+			(effects
+				(font
