File: KICAD/MP3_Player/audio.kicad_sch (KiCad schematic)
At the start: 23 parts, among them J7 AudioPlug4, J8 AudioPlug4, U6 PCM5102AQPWRQ1

Commit message: Add files via upload
Parts:
- renumbered CAPM to C45
Connections:
- net CODEC_BCK renamed DAC_BCK
- net CODEC_DIN renamed DAC_DIN
- net CODEC_LRCK renamed DAC_LRCK
- net CODEC_XSMT renamed DAC_XSMT
Other:
- note added: "I2S DAC"
- note removed: "I2S CODEC"
- moved on the sheet: C43, C44, C45
Changed lines of the file:
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@@
 		)
 	)
-	(text "I2S CODEC"
+	(text "I2S DAC"
 		(exclude_from_sim no)
 		(at 156.972 123.444 0)
@@
 	)
 	(junction
-		(at 198.12 67.31)
+		(at 203.2 67.31)
 		(diameter 0)
 		(color 0 0 0 0)
@@
 	)
 	(junction
-		(at 198.12 81.28)
+		(at 203.2 81.28)
 		(diameter 0)
 		(color 0 0 0 0)
@@
 	)
 	(junction
-		(at 186.69 69.85)
+		(at 191.77 69.85)
 		(diameter 0)
 		(color 0 0 0 0)
@@
 	(wire
 		(pts
-			(xy 198.12 80.01) (xy 198.12 81.28)
+			(xy 203.2 80.01) (xy 203.2 81.28)
 		)
 		(stroke
@@
 	(wire
 		(pts
-			(xy 209.55 69.85) (xy 186.69 69.85)
-		)
-		(stroke
-			(width 0)
-			(type default)
-		)
-	)
-	(wire
-		(pts
 			(xy 58.42 147.32) (xy 58.42 151.13)
 		)
@@
 	(wire
 		(pts
-			(xy 166.37 87.63) (xy 168.91 87.63)
-		)
-		(stroke
-			(width 0)
-			(type default)
-		)
-	)
-	(wire
-		(pts
-			(xy 198.12 81.28) (xy 213.36 81.28)
+			(xy 166.37 87.63) (xy 170.18 87.63)
 		)
 		(stroke
@@
 	(wire
 		(pts
-			(xy 166.37 95.25) (xy 168.91 95.25)
+			(xy 166.37 95.25) (xy 170.18 95.25)
 		)
 		(stroke
@@
 	(wire
 		(pts
-			(xy 186.69 69.85) (xy 181.61 69.85)
+			(xy 181.61 69.85) (xy 209.55 69.85)
 		)
 		(stroke
@@
 	(wire
 		(pts
-			(xy 198.12 67.31) (xy 217.17 67.31)
-		)
-		(stroke
-			(width 0)
-			(type default)
-		)
-	)
-	(wire
-		(pts
 			(xy 151.13 62.23) (xy 156.21 62.23)
 		)
@@
 	(wire
 		(pts
-			(xy 198.12 67.31) (xy 198.12 72.39)
+			(xy 203.2 67.31) (xy 203.2 72.39)
 		)
 		(stroke
@@
 	(wire
 		(pts
-			(xy 186.69 69.85) (xy 186.69 72.39)
+			(xy 191.77 69.85) (xy 191.77 72.39)
 		)
 		(stroke
@@
 	(wire
 		(pts
-			(xy 186.69 81.28) (xy 198.12 81.28)
+			(xy 191.77 81.28) (xy 213.36 81.28)
 		)
 		(stroke
@@
 	(wire
 		(pts
-			(xy 186.69 80.01) (xy 186.69 81.28)
+			(xy 191.77 80.01) (xy 191.77 81.28)
 		)
 		(stroke
@@
 	(wire
 		(pts
-			(xy 179.07 67.31) (xy 198.12 67.31)
+			(xy 179.07 67.31) (xy 217.17 67.31)
 		)
 		(stroke
@@
 		)
 	)
-	(hierarchical_label "CODEC_XSMT"
+	(hierarchical_label "DAC_XSMT"
 		(shape input)
 		(at 132.08 97.79 180)
@@
 		)
 	)
-	(hierarchical_label "CODEC_LRCK"
+	(hierarchical_label "DAC_LRCK"
 		(shape input)
 		(at 132.08 80.01 180)
@@
 		)
 	)
-	(hierarchical_label "CODEC_DIN"
+	(hierarchical_label "DAC_DIN"
 		(shape input)
 		(at 132.08 82.55 180)
@@
 		)
 	)
-	(hierarchical_label "CODEC_BCK"
+	(hierarchical_label "DAC_BCK"
 		(shape input)
 		(at 132.08 85.09 180)
@@
 	(symbol
 		(lib_id "Device:C")
-		(at 186.69 76.2 0)
+		(at 191.77 76.2 0)
 		(unit 1)
 		(body_style 1)
@@
 		(fields_autoplaced yes)
 		(property "Reference" "C43"
-			(at 190.5 74.9299 0)
+			(at 195.58 74.9299 0)
 			(show_name no)
 			(do_not_autoplace no)
@@
 		)
 		(property "Value" "2n2"
-			(at 190.5 77.4699 0)
+			(at 195.58 77.4699 0)
 			(show_name no)
 			(do_not_autoplace no)
@@
 		)
 		(property "Footprint" ""
-			(at 187.6552 80.01 0)
+			(at 192.7352 80.01 0)
 			(hide yes)
 			(show_name no)
@@
 		)
 		(property "Datasheet" ""
-			(at 186.69 76.2 0)
+			(at 191.77 76.2 0)
 			(hide yes)
 			(show_name no)
@@
 		)
 		(property "Description" "Unpolarized capacitor"
-			(at 186.69 76.2 0)
+			(at 191.77 76.2 0)
 			(hide yes)
 			(show_name no)
@@
 	(symbol
 		(lib_id "Device:C")
-		(at 168.91 91.44 0)
+		(at 170.18 91.44 0)
 		(unit 1)
 		(body_style 1)
@@
 		(dnp no)
 		(fields_autoplaced yes)
-		(property "Reference" "CAPM"
-			(at 172.72 90.1699 0)
+		(property "Reference" "C45"
+			(at 173.99 90.1699 0)
 			(show_name no)
 			(do_not_autoplace no)
@@
 		)
 		(property "Value" "2u2"
-			(at 172.72 92.7099 0)
+			(at 173.99 92.7099 0)
 			(show_name no)
 			(do_not_autoplace no)
@@
 		)
 		(property "Footprint" ""
-			(at 169.8752 95.25 0)
+			(at 171.1452 95.25 0)
 			(hide yes)
 			(show_name no)
@@
 		)
 		(property "Datasheet" ""
-			(at 168.91 91.44 0)
+			(at 170.18 91.44 0)
 			(hide yes)
 			(show_name no)
@@
 		)
 		(property "Description" "Unpolarized capacitor"
-			(at 168.91 91.44 0)
+			(at 170.18 91.44 0)
 			(hide yes)
 			(show_name no)
@@
 			(project "MP3_Player"
 				(path "/5963f475-7f70-4482-9734-331d34890960/31a039c0-b270-42d0-8a83-cc75fb8b1933"
-					(reference "CAPM")
+					(reference "C45")
 					(unit 1)
 				)
@@
 	(symbol
 		(lib_id "Device:C")
-		(at 198.12 76.2 0)
+		(at 203.2 76.2 0)
 		(unit 1)
 		(body_style 1)
@@
 		(fields_autoplaced yes)
 		(property "Reference" "C44"
-			(at 201.93 74.9299 0)
+			(at 207.01 74.9299 0)
 			(show_name no)
 			(do_not_autoplace no)
@@
 		)
 		(property "Value" "2n2"
-			(at 201.93 77.4699 0)
+			(at 207.01 77.4699 0)
 			(show_name no)
 			(do_not_autoplace no)
@@
 		)
 		(property "Footprint" ""
-			(at 199.0852 80.01 0)
+			(at 204.1652 80.01 0)
 			(hide yes)
 			(show_name no)
@@
 		)
 		(property "Datasheet" ""
-			(at 198.12 76.2 0)
+			(at 203.2 76.2 0)
 			(hide yes)
 			(show_name no)
@@
 		)
 		(property "Description" "Unpolarized capacitor"
-			(at 198.12 76.2 0)
+			(at 203.2 76.2 0)
 			(hide yes)
 			(show_name no)
@@
 		(in_pos_files yes)
 		(dnp no)
-		(fields_autoplaced yes)
 		(property "Reference" "U6"
-			(at 158.3533 72.39 0)
+			(at 158.496 69.85 0)
 			(show_name no)
 			(do_not_autoplace no)
@@
 		)
 		(property "Value" "PCM5102AQPWRQ1"
-			(at 158.3533 74.93 0)
+			(at 158.496 72.39 0)
 			(show_name no)
 			(do_not_autoplace no)
