File: KICAD/MP3_Player/mcu.kicad_sch (KiCad schematic)
At the start: 25 parts, among them J1 TC2030, J4 Conn_01x03_Pin, U1 STM32F411CEU6, U8 PCAL6408ABSHP, Y1 25MHz, Y2 32.768KHz

Commit message: Add files via upload
Parts:
- removed J4: Conn_01x03_Pin, symbol Connector:Conn_01x03_Pin
- removed R8: 0r, symbol Device:R
- added JP2, JP3: Boot Select, symbol Jumper:SolderJumper_3_Bridged12
- added TP10: SDA, symbol Connector:TestPoint
- added TP7: HSE, symbol Connector:TestPoint
- added TP8: LSE, symbol Connector:TestPoint
- added TP9: SCL, symbol Connector:TestPoint
Connections:
- net +3V3: now also JP2.1 (A), JP3.3 (B)
- net BOOT0R: now also JP2.2 (C)
- net GND: now also JP2.3 (B), JP3.1 (A); no longer U8.16 (ADDR)
- net HSE_OUT: now also TP7.1
- net LSE_OUT: now also TP8.1
- net SCL: now also TP9.1
- net SDA: now also TP10.1
- net MUX_INT: now reaches U1.2 (PC13)
- net MUX_INT: now also U8.11 (~{INT})
- net CODEC_BCK renamed DAC_BCK
- net CODEC_DIN renamed DAC_DIN
- net CODEC_LRCK renamed DAC_LRCK
- net CODEC_XSMT renamed DAC_XSMT
- new net: JP3.2 (C), U8.16 (ADDR)
- no-connect marks 2 -> 0
Other:
- note added: "Enable pull-ups for buttons in frimware"
- note added: "I2C Test Points"
- note added: "Only cut and bridge once MCU firmware is done"
- note removed: "Only place once MCU Firmware is done"
