File: KICAD/MP3_Player/power.kicad_sch (KiCad schematic)
At the start: 14 parts, among them J5 BAT Connector, SW1 Power SW, U2 AP2112K-3.3, U3 BQ24075RGTR, U5 MAX17048G

Commit message: Add files via upload
Parts:
- added TP3: BAT, Relay_THT:Relay_DPDT_Schrack-RT2-FormC_RM5mm, symbol Connector:TestPoint
- added TP4: GND, Relay_THT:Relay_DPDT_Schrack-RT2-FormC_RM5mm, symbol Connector:TestPoint
- added TP5: BQ_OUT, Relay_THT:Relay_DPDT_Schrack-RT2-FormC_RM5mm, symbol Connector:TestPoint
- added TP6: +3V3, Relay_THT:Relay_DPDT_Schrack-RT2-FormC_RM5mm, symbol Connector:TestPoint
- R10: value 4k7 -> 1k
Connections:
- net +VBAT: now also U3.6 (EN1), TP6.1
- net BAT +: now also TP3.1
- net BAT_OUT: now also TP5.1; no longer U3.6 (EN1)
- net GND: now also TP4.1
Other:
- note added: "For ERC Ignore"
- moved on the sheet: C14, R10
