File: KICAD/MP3_Player/wireless.kicad_sch (KiCad schematic)
At the start: 10 parts, among them U7 ST67W611M1A6B, Y3 32.768KHz

Commit message: Add files via upload
Parts:
- added JP1: Boot Select, symbol Jumper:SolderJumper_2_Open
- added R25: 10k, symbol Device:R
- added TP1: UART_TX, Relay_THT:Relay_DPDT_Schrack-RT2-FormC_RM5mm, symbol Connector:TestPoint
- added TP2: UART_RX, Relay_THT:Relay_DPDT_Schrack-RT2-FormC_RM5mm, symbol Connector:TestPoint
Connections:
- net +3V3: now also JP1.2 (B)
- net Chip_EN: now also C34.2; no longer C34.1
- net GND: now also C34.1, R25.2; no longer C34.2, U7.3 (BOOT)
- net at U7.22 (UART_TX): now also TP1.1
- net at U7.23 (UART_RX): now also TP2.1
- net W_XTALIN: no longer names the net of C32.1, U7.14 (XTAL32K_IN), Y3.1
- net W_XTALOUT: no longer names the net of C33.1, U7.13 (XTAL32K_OUT), Y3.2
- new net: JP1.1 (A), R25.1, U7.3 (BOOT)
- no-connect marks 3 -> 1
Other:
- moved on the sheet: R16
