File: PCB/MP3_Player/MP3_Player.kicad_sch (KiCad schematic)
At the start: 0 parts

Commit message: Minor Schematic Changes
Changed lines of the file:
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@@
+	(wire
+		(pts
+			(xy 166.37 120.65) (xy 218.44 120.65)
+		)
+		(stroke
+			(width 0)
+			(type default)
+		)
+	)
+	(wire
+		(pts
+			(xy 113.03 166.37) (xy 148.59 166.37)
+		)
+		(stroke
+			(width 0)
+			(type default)
+		)
+	)
+	(wire
+		(pts
+			(xy 166.37 85.09) (xy 218.44 85.09)
+		)
+		(stroke
+			(width 0)
+			(type default)
+		)
+	)
+	(wire
+		(pts
+			(xy 74.93 76.2) (xy 137.16 76.2)
+		)
+		(stroke
+			(width 0)
+			(type default)
+		)
+	)
+	(wire
+		(pts
+			(xy 166.37 44.45) (xy 218.44 44.45)
+		)
+		(stroke
+			(width 0)
+			(type default)
+		)
+	)
+	(wire
+		(pts
+			(xy 113.03 171.45) (xy 153.67 171.45)
+		)
+		(stroke
+			(width 0)
+			(type default)
+		)
+	)
+	(wire
+		(pts
+			(xy 148.59 166.37) (xy 148.59 138.43)
+		)
+		(stroke
+			(width 0)
+			(type default)
+		)
+	)
 	(wire
 		(pts
@@
 	(wire
 		(pts
-			(xy 166.37 120.65) (xy 218.44 120.65)
-		)
-		(stroke
-			(width 0)
-			(type default)
-		)
-	)
-	(wire
-		(pts
-			(xy 166.37 85.09) (xy 218.44 85.09)
-		)
-		(stroke
-			(width 0)
-			(type default)
-		)
-	)
-	(wire
-		(pts
-			(xy 74.93 76.2) (xy 137.16 76.2)
-		)
-		(stroke
-			(width 0)
-			(type default)
-		)
-	)
-	(wire
-		(pts
-			(xy 166.37 44.45) (xy 218.44 44.45)
-		)
-		(stroke
-			(width 0)
-			(type default)
-		)
-	)
-	(wire
-		(pts
-			(xy 113.03 171.45) (xy 153.67 171.45)
-		)
-		(stroke
-			(width 0)
-			(type default)
-		)
-	)
-	(wire
-		(pts
 			(xy 166.37 41.91) (xy 218.44 41.91)
 		)
@@
 	(wire
 		(pts
-			(xy 148.59 166.37) (xy 148.59 133.35)
-		)
-		(stroke
-			(width 0)
-			(type default)
-		)
-	)
-	(wire
-		(pts
 			(xy 74.93 39.37) (xy 137.16 39.37)
 		)
@@
 	(wire
 		(pts
-			(xy 113.03 166.37) (xy 148.59 166.37)
-		)
-		(stroke
-			(width 0)
-			(type default)
-		)
-	)
-	(wire
-		(pts
 			(xy 166.37 118.11) (xy 218.44 118.11)
 		)
@@
 	(wire
 		(pts
-			(xy 153.67 171.45) (xy 153.67 133.35)
+			(xy 153.67 171.45) (xy 153.67 138.43)
 		)
 		(stroke
@@
 	(wire
 		(pts
-			(xy 156.21 133.35) (xy 156.21 173.99)
+			(xy 156.21 138.43) (xy 156.21 173.99)
 		)
 		(stroke
@@
 		)
 		(pin "+VBAT" bidirectional
-			(at 148.59 133.35 270)
+			(at 148.59 138.43 270)
 			(effects
 				(font
@@
 		)
 		(pin "SCL" output
-			(at 153.67 133.35 270)
+			(at 153.67 138.43 270)
 			(effects
 				(font
@@
 		)
 		(pin "SDA" bidirectional
-			(at 156.21 133.35 270)
-			(effects
-				(font
+			(at 156.21 138.43 270)
+			(effects
+				(font
