File: PCB/MP3_Player/mcu.kicad_sch (KiCad schematic)
At the start: 29 parts, among them J1 TC2030, U1 STM32F411CEU6, U8 PCAL6408ABSHP, Y1 25MHz, Y2 32.768KHz

Commit message: Minor Schematic Changes
Other:
- note added: "Change if it has address conflicts"
Changed lines of the file:
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@@
+		)
+	)
+	(text "Change if it has\naddress conflicts"
+		(exclude_from_sim no)
+		(at 39.878 169.926 0)
+		(effects
+			(font
+				(size 1.27 1.27)
+			)
 		)
 	)

Commit message: Visual Schematic Corrections
Other:
- note added: "Cut and bridge once MCU firmware is done"
- note removed: "Only cut and bridge once MCU firmware is done"
Changed lines of the file:
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@@
 		)
 	)
-	(text "Only cut and bridge once \n  MCU firmware is done"
+	(text "Cut and bridge once MCU\nfirmware is done"
 		(exclude_from_sim no)
-		(at 23.622 90.424 0)
+		(at 31.496 94.488 0)
 		(effects
 			(font
 				(size 1.27 1.27)
 			)
-			(justify left)
 		)
 	)

Commit message: Started Making BOM
Parts:
- C1, C2, C3, C37, C38, C4, C6: Mfr. Part # (none) -> CL05B104KP5NNNC; Store URL - Digikey (none) -> https://www.digikey.pt/pt/products/detail/samsung-electro-m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; Store URL - Mouser (none) -> https://pt.mouser.com/en/ProductDetail/Samsung-Electro-Mech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
- C10, C11, C12, C9: Mfr. Part # (none) -> CL05C2R2CB51PNC; Store URL - Digikey (none) -> https://www.digikey.pt/pt/products/detail/samsung-electro-m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; Store URL - Mouser (none) -> https://pt.mouser.com/en/ProductDetail/Samsung-Electro-Mech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
- C5: Mfr. Part # (none) -> CL10A106KP8NNNC; Store URL - Digikey (none) -> https://www.digikey.pt/pt/products/detail/samsung-electro-m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; Store URL - Mouser (none) -> https://pt.mouser.com/en/ProductDetail/Samsung-Electro-Mech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
- C7: Mfr. Part # (none) -> CL05A105MQ5NNND; Store URL - Digikey (none) -> https://www.digikey.pt/pt/products/detail/samsung-electro-m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; Store URL - Mouser (none) -> https://pt.mouser.com/en/ProductDetail/Samsung-Electro-Mech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
- C8: Mfr. Part # (none) -> NMC0603X5R475K6.3TRPF; Store URL - Digikey (none) -> https://www.digikey.pt/pt/products/detail/nic-components-co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
- TP10, TP7, TP8, TP9: now left out of the parts list

Commit message: Continue Making BOM
Parts:
- FB1: Mfr. Part # (none) -> BLM15AG601SN1D; Store URL - Digikey (none) -> https://www.digikey.pt/pt/products/detail/murata-electronic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; Store URL - Mouser (none) -> https://pt.mouser.com/en/ProductDetail/Murata-Electronics/B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
- R1: Mfr. Part # (none) -> CRCW040210K0FKED; Store URL - Digikey (none) -> https://www.digikey.pt/pt/products/detail/vishay-dale/CRCW0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; Store URL - Mouser (none) -> https://pt.mouser.com/en/ProductDetail/Vishay/CRCW040210K0F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
- R14, R15: Mfr. Part # (none) -> CRCW04024K70FKED; Store URL - Digikey (none) -> https://www.digikey.pt/pt/products/detail/vishay-dale/CRCW0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; Store URL - Mouser (none) -> https://pt.mouser.com/en/ProductDetail/Vishay/CRCW04024K70F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
Changed lines of the file:
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@@
 			)
 		)
-		(property "Datasheet" ""
+		(property "Datasheet" "https://pim.murata.com/asset/pim4/ferriteBeadInductortypefilter/ENFA0018_PDF_FERRITEBEADINDUCTORTYPEFILTER?lastModifiedDatetime=20250707191428"
 			(at 200.66 45.72 0)
 			(hide yes)
@@
 			)
 		)
-		(property "Description" "Ferrite bead"
+		(property "Description" "0402"
 			(at 200.66 45.72 0)
 			(hide yes)
@@
 		)
 		(property "Store URL - TME" ""
+			(at 200.66 45.72 90)
+			(hide yes)
+			(show_name no)
+			(do_not_autoplace no)
+			(effects
+				(font
+					(size 1.27 1.27)
+				)
+			)
+		)
+		(property "Mfr. Part #" "BLM15AG601SN1D"
+			(at 200.66 45.72 90)
+			(hide yes)
+			(show_name no)
+			(do_not_autoplace no)
+			(effects
+				(font
+					(size 1.27 1.27)
+				)
+			)
+		)
+		(property "Store URL - Digikey" "https://www.digikey.pt/pt/products/detail/murata-electronics/BLM15AG601SN1D/584217"
+			(at 200.66 45.72 90)
+			(hide yes)
+			(show_name no)
+			(do_not_autoplace no)
+			(effects
+				(font
+					(size 1.27 1.27)
+				)
+			)
+		)
+		(property "Store URL - Mouser" "https://pt.mouser.com/en/ProductDetail/Murata-Electronics/BLM15AG601SN1D?qs=%2FjCH2pcB5WLSIF5DG9Nbqw%3D%3D"
 			(at 200.66 45.72 90)
 			(hide yes)
@@
 			)
 		)
-		(property "Datasheet" ""
+		(property "Datasheet" "https://www.vishay.com/docs/20035/dcrcwe3.pdf"
 			(at 64.77 87.63 0)
 			(hide yes)
@@
 			)
 		)
-		(property "Description" "Resistor"
+		(property "Description" "0402"
 			(at 64.77 87.63 0)
 			(hide yes)
@@
 		)
 		(property "Store URL - TME" ""
+			(at 64.77 87.63 90)
+			(hide yes)
+			(show_name no)
+			(do_not_autoplace no)
+			(effects
+				(font
+					(size 1.27 1.27)
+				)
+			)
+		)
+		(property "Mfr. Part #" "CRCW040210K0FKED"
+			(at 64.77 87.63 90)
+			(hide yes)
+			(show_name no)
+			(do_not_autoplace no)
+			(effects
+				(font
+					(size 1.27 1.27)
+				)
+			)
+		)
+		(property "Store URL - Digikey" "https://www.digikey.pt/pt/products/detail/vishay-dale/CRCW040210K0FKED/1178121"
+			(at 64.77 87.63 90)
+			(hide yes)
+			(show_name no)
+			(do_not_autoplace no)
+			(effects
+				(font
+					(size 1.27 1.27)
+				)
+			)
+		)
+		(property "Store URL - Mouser" "https://pt.mouser.com/en/ProductDetail/Vishay/CRCW040210K0FKED?qs=rlE3Te1NifyN3e8vvxacSw%3D%3D"
 			(at 64.77 87.63 90)
 			(hide yes)
@@
 			)
 		)
-		(property "Datasheet" ""
+		(property "Datasheet" "https://www.vishay.com/docs/20035/dcrcwe3.pdf"
 			(at 58.42 153.67 0)
 			(hide yes)
@@
 			)
 		)
-		(property "Description" "Resistor"
+		(property "Description" "0402"
 			(at 58.42 153.67 0)
 			(hide yes)
@@
 		)
 		(property "Store URL - TME" ""
+			(at 58.42 153.67 0)
+			(hide yes)
+			(show_name no)
+			(do_not_autoplace no)
+			(effects
+				(font
+					(size 1.27 1.27)
+				)
+			)
+		)
+		(property "Mfr. Part #" "CRCW04024K70FKED"
+			(at 58.42 153.67 0)
+			(hide yes)
+			(show_name no)
+			(do_not_autoplace no)
+			(effects
+				(font
+					(size 1.27 1.27)
+				)
+			)
+		)
+		(property "Store URL - Digikey" "https://www.digikey.pt/pt/products/detail/vishay-dale/CRCW04024K70FKED/1178083"
+			(at 58.42 153.67 0)
+			(hide yes)
+			(show_name no)
+			(do_not_autoplace no)
+			(effects
+				(font
+					(size 1.27 1.27)
+				)
+			)
+		)
+		(property "Store URL - Mouser" "https://pt.mouser.com/en/ProductDetail/Vishay/CRCW04024K70FKED?qs=Jz%252BxJjKhzTxI08uguE%252B9mA%3D%3D"
 			(at 58.42 153.67 0)
 			(hide yes)
@@
 			)
 		)
-		(property "Datasheet" ""
+		(property "Datasheet" "https://www.vishay.com/docs/20035/dcrcwe3.pdf"
 			(at 50.8 153.67 0)
 			(hide yes)
@@
 			)
 		)
-		(property "Description" "Resistor"
+		(property "Description" "0402"
 			(at 50.8 153.67 0)
 			(hide yes)
@@
 			(at 50.8 153.67 0)
 			(hide yes)
+			(show_name no)
+			(do_not_autoplace no)
+			(effects
+				(font
+					(size 1.27 1.27)
+				)
+			)
+		)
+		(property "Mfr. Part #" "CRCW04024K70FKED"
+			(at 50.8 153.67 0)
+			(hide yes)
+			(show_name no)
+			(do_not_autoplace no)
+			(effects
+				(font
+					(size 1.27 1.27)
+				)
+			)
+		)
+		(property "Store URL - Digikey" "https://www.digikey.pt/pt/products/detail/vishay-dale/CRCW04024K70FKED/1178083"
+			(at 50.8 153.67 0)
+			(hide yes)
+			(show_name no)
+			(do_not_autoplace no)
+			(effects
+				(font
+					(size 1.27 1.27)
+				)
+			)
+		)
+		(property "Store URL - Mouser" "https://pt.mouser.com/en/ProductDetail/Vishay/CRCW04024K70FKED?qs=Jz%252BxJjKhzTxI08uguE%252B9mA%3D%3D"
+			(at 50.8 153.67 0)
+			(hide yes)

Commit message: Finished BOM; Started Footprint assignment
Parts:
- C1, C10, C11, C12, C2, C3, C37, C38, C4, C6, C7, C9, FB1, R1, R14, R15: footprint (none) -> Capacitor_SMD:C_0402_1005Metric
- C5: footprint (none) -> Capacitor_SMD:C_0603_1608Metric
- C8: footprint (none) -> Capacitor_SMD:C_0603_1608Metric; Mfr. Part # NMC0603X5R475K6.3TRPF -> CL10A475KA8NQNC; Store URL - Digikey https://www.digikey.pt/pt/products/detail/nic-components-co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 -> https://www.digikey.pt/pt/products/detail/samsung-electro-m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; Store URL - Mouser (none) -> https://pt.mouser.com/en/ProductDetail/Samsung-Electro-Mech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
Changed lines of the file:
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@@
 			)
 		)
-		(property "Footprint" ""
+		(property "Footprint" "Capacitor_SMD:C_0402_1005Metric"
 			(at 168.6052 40.64 0)
 			(hide yes)
@@
 			)
 		)
-		(property "Footprint" ""
+		(property "Footprint" "Capacitor_SMD:C_0603_1608Metric"
 			(at 145.7452 40.64 0)
 			(hide yes)
@@
 			)
 		)
-		(property "Footprint" ""
+		(property "Footprint" "Capacitor_SMD:C_0402_1005Metric"
 			(at 157.1752 40.64 0)
 			(hide yes)
@@
 			)
 		)
-		(property "Footprint" ""
+		(property "Footprint" "Capacitor_SMD:C_0402_1005Metric"
 			(at 126.0348 123.19 0)
 			(hide yes)
@@
 			)
 		)
-		(property "Footprint" ""
+		(property "Footprint" "Capacitor_SMD:C_0402_1005Metric"
 			(at 213.0552 55.88 0)
 			(hide yes)
@@
 			)
 		)
-		(property "Footprint" ""
+		(property "Footprint" "Capacitor_SMD:C_0402_1005Metric"
 			(at 140.6652 96.52 0)
 			(hide yes)
@@
 			)
 		)
-		(property "Footprint" ""
+		(property "Footprint" "Capacitor_SMD:C_0402_1005Metric"
 			(at 180.0352 40.64 0)
 			(hide yes)
@@
 			)
 		)
-		(property "Footprint" ""
+		(property "Footprint" "Capacitor_SMD:C_0603_1608Metric"
 			(at 168.6052 148.59 0)
 			(hide yes)
@@
 			)
 		)
-		(property "Datasheet" "https://www.niccomp.com/wp-content/uploads/catalog/nmchc.pdf"
+		(property "Datasheet" "https://mm.digikey.com/Volume0/opasdata/d220001/medias/docus/43/CL10A475KA8NQNC_Spec.pdf"
 			(at 167.64 144.78 0)
 			(hide yes)
@@
 			)
 		)
-		(property "Mfr. Part #" "NMC0603X5R475K6.3TRPF"
+		(property "Mfr. Part #" "CL10A475KA8NQNC"
+			(at 167.64 144.78 0)
+			(hide yes)
+			(show_name no)
+			(do_not_autoplace no)
+			(effects
+				(font
+					(size 1.27 1.27)
+				)
+			)
+		)
+		(property "Store URL - Digikey" "https://www.digikey.pt/pt/products/detail/samsung-electro-mechanics/CL10A475KA8NQNC/3887558?s=N4IgTCBcDaIMIBkCMAGAggFgOwFYDSaAHAHICKxcIAugL5A"
 			(at 167.64 144.78 0)
 			(hide yes)
@@
 			)
 		)
-		(property "Store URL - Digikey" "https://www.digikey.pt/pt/products/detail/nic-components-corp/NMC0603X5R475K6-3TRPF/18896085?s=N4IgjCBcoKxaBjKAzAhgGwM4FMA0IB7KAbRABYBOCgdhgAYQBdfABwBcoQBlNgJwEsAdgHMQAX3xgAbPBBJIaLHkIkQAZgoAmMjOYh2nHgJHjJFABwVZ8xTnxFIpBowkhNdStZQY7Kx%2BQA6agACAFaAMSZWDkgQAFVBfjYAeWQAWWxUTABXXmxxMTEgA"
+		(property "Store URL - Mouser" "https://pt.mouser.com/en/ProductDetail/Samsung-Electro-Mechanics/CL10A475KA8NQNC?qs=9nYkJLYMUzsiOkP%2FacWBkg%3D%3D"
 			(at 167.64 144.78 0)
 			(hide yes)
@@
 			)
 		)
-		(property "Footprint" ""
+		(property "Footprint" "Capacitor_SMD:C_0402_1005Metric"
 			(at 200.66 47.498 90)
 			(hide yes)
@@
 			)
 		)
-		(property "Footprint" ""
+		(property "Footprint" "Capacitor_SMD:C_0402_1005Metric"
 			(at 224.4852 55.88 0)
 			(hide yes)
@@
 			)
 		)
-		(property "Footprint" ""
+		(property "Footprint" "Capacitor_SMD:C_0402_1005Metric"
 			(at 87.3252 148.59 0)
 			(hide yes)
@@
 			)
 		)
-		(property "Footprint" ""
+		(property "Footprint" "Capacitor_SMD:C_0402_1005Metric"
 			(at 140.6652 123.19 0)
 			(hide yes)
@@
 			)
 		)
-		(property "Footprint" ""
+		(property "Footprint" "Capacitor_SMD:C_0402_1005Metric"
 			(at 126.0348 96.52 0)
 			(hide yes)
@@
 			)
 		)
-		(property "Footprint" ""
+		(property "Footprint" "Capacitor_SMD:C_0402_1005Metric"
 			(at 64.77 89.408 90)
 			(hide yes)
@@
 			)
 		)
-		(property "Footprint" ""
+		(property "Footprint" "Capacitor_SMD:C_0402_1005Metric"
 			(at 56.642 153.67 90)
 			(hide yes)
@@
 			)
 		)
-		(property "Footprint" ""
+		(property "Footprint" "Capacitor_SMD:C_0402_1005Metric"
 			(at 160.9852 63.5 0)
 			(hide yes)
@@
 			)
 		)
-		(property "Footprint" ""
+		(property "Footprint" "Capacitor_SMD:C_0402_1005Metric"
 			(at 100.0252 148.59 0)
 			(hide yes)
@@
 			)
 		)
-		(property "Footprint" ""
+		(property "Footprint" "Capacitor_SMD:C_0402_1005Metric"
 			(at 49.022 153.67 90)
 			(hide yes)

Commit message: Footprint Assingment
Parts:
- JP2: footprint (none) -> Jumper:SolderJumper-3_P1.3mm_Bridged12_RoundedPad1.0x1.5mm
- JP3: value Boot Select -> Addr Select; footprint (none) -> Jumper:SolderJumper-3_P1.3mm_Bridged12_RoundedPad1.0x1.5mm
- R1, R14, R15: footprint Capacitor_SMD:C_0402_1005Metric -> Resistor_SMD:R_0402_1005Metric
- TP10, TP7, TP8, TP9: footprint (none) -> TestPoint:TestPoint_Pad_D1.5mm
Changed lines of the file:
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@@
 			)
 		)
-		(property "Footprint" ""
+		(property "Footprint" "TestPoint:TestPoint_Pad_D1.5mm"
 			(at 152.4 76.2 0)
 			(hide yes)
@@
 			)
 		)
-		(property "Footprint" ""
+		(property "Footprint" "TestPoint:TestPoint_Pad_D1.5mm"
 			(at 252.73 35.56 0)
 			(hide yes)
@@
 			)
 		)
-		(property "Footprint" ""
+		(property "Footprint" "Jumper:SolderJumper-3_P1.3mm_Bridged12_RoundedPad1.0x1.5mm"
 			(at 50.8 95.25 0)
 			(hide yes)
@@
 			)
 		)
-		(property "Value" "Boot Select"
+		(property "Value" "Addr Select"
 			(at 48.26 177.7999 90)
 			(show_name no)
@@
 			)
 		)
-		(property "Footprint" ""
+		(property "Footprint" "Jumper:SolderJumper-3_P1.3mm_Bridged12_RoundedPad1.0x1.5mm"
 			(at 50.8 176.53 0)
 			(hide yes)
@@
 			)
 		)
-		(property "Footprint" ""
+		(property "Footprint" "TestPoint:TestPoint_Pad_D1.5mm"
 			(at 252.73 38.1 0)
 			(hide yes)
@@
 			)
 		)
-		(property "Footprint" "Capacitor_SMD:C_0402_1005Metric"
+		(property "Footprint" "Resistor_SMD:R_0402_1005Metric"
 			(at 64.77 89.408 90)
 			(hide yes)
@@
 			)
 		)
-		(property "Footprint" ""
+		(property "Footprint" "TestPoint:TestPoint_Pad_D1.5mm"
 			(at 161.29 76.2 0)
 			(hide yes)
@@
 			)
 		)
-		(property "Footprint" "Capacitor_SMD:C_0402_1005Metric"
+		(property "Footprint" "Resistor_SMD:R_0402_1005Metric"
 			(at 56.642 153.67 90)
 			(hide yes)
@@
 			)
 		)
-		(property "Footprint" "Capacitor_SMD:C_0402_1005Metric"
+		(property "Footprint" "Resistor_SMD:R_0402_1005Metric"
 			(at 49.022 153.67 90)
 			(hide yes)

Commit message: Footprint Assingment Complete
Parts:
- TP10, TP7, TP8, TP9: footprint TestPoint:TestPoint_Pad_D1.5mm -> TestPoint:TestPoint_Pad_D1.0mm
Changed lines of the file:
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@@
 			)
 		)
-		(property "Footprint" "TestPoint:TestPoint_Pad_D1.5mm"
+		(property "Footprint" "TestPoint:TestPoint_Pad_D1.0mm"
 			(at 152.4 76.2 0)
 			(hide yes)
@@
 			)
 		)
-		(property "Footprint" "TestPoint:TestPoint_Pad_D1.5mm"
+		(property "Footprint" "TestPoint:TestPoint_Pad_D1.0mm"
 			(at 252.73 35.56 0)
 			(hide yes)
@@
 			)
 		)
-		(property "Footprint" "TestPoint:TestPoint_Pad_D1.5mm"
+		(property "Footprint" "TestPoint:TestPoint_Pad_D1.0mm"
 			(at 252.73 38.1 0)
 			(hide yes)
@@
 			)
 		)
-		(property "Footprint" "TestPoint:TestPoint_Pad_D1.5mm"
+		(property "Footprint" "TestPoint:TestPoint_Pad_D1.0mm"
 			(at 161.29 76.2 0)
 			(hide yes)

Commit message: Starting PCB Layout
Connections:
- net ADDR_SELECT: now reaches JP3.2 (C), U8.16 (ADDR)
Changed lines of the file:
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@@
+		)
+	)
+	(label "ADDR_SELECT"
+		(at 54.61 176.53 0)
+		(effects
+			(font
+				(size 1.27 1.27)
+			)
+			(justify left bottom)
 		)
 	)
