File: PCB/MP3_Player/mcu.kicad_sch (KiCad schematic)
At the start: 29 parts, among them J1 TC2030, U1 STM32F411CEU6, U8 PCAL6408ABSHP, Y1 25MHz, Y2 32.768KHz

Commit message: PCB Routing
Connections:
- net B_Down: now also U8.4 (P2); no longer U8.3 (P1)
- net B_Left: now also U8.3 (P1); no longer U8.4 (P2)
- net B_Ok: now also U8.5 (P3); no longer U8.7 (P4)
- net B_Right: now also U8.7 (P4); no longer U8.5 (P3)
