File: PCB/MP3_Player/usb.kicad_sch (KiCad schematic)
At the start: 13 parts, among them J2 USB_C_Receptacle_16P, J3 USB_A, U4 TS3USB30ERSWR

Commit message: PCB Routing
Parts:
- removed U4: TS3USB30ERSWR, Package_DFN_QFN:UQFN-10_1.4x1.8mm_P0.4mm, symbol Interface_USB:TS3USB30ERSWR
- added IC1: TS3USB221AQRSERQ1, TS3USB221AQRSERQ1:TS3USB221AQRSERQ1, symbol TS3USB221AQRSERQ1:TS3USB221AQRSERQ1
Connections:
- net +3V3: now also IC1.10 (VCC)
- net D+: now also IC1.8 (D+)
- net D-: now also IC1.7 (D-)
- net GND: now also IC1.5 (GND), IC1.6 (~{OE})
- net Output SW: now also IC1.9 (S)
- net USB-A_DN: now also IC1.4 (2D-)
- net USB-A_DP: now also IC1.3 (2D+)
- net USB-C_DN: now also IC1.2 (1D-)
- net USB-C_DP: now also IC1.1 (1D+)
Other:
- moved on the sheet: C13, R8

Commit message: PCB Routing
Connections:
- net USB-A_DN: now also IC1.2 (1D-); no longer IC1.4 (2D-)
- net USB-A_DP: now also IC1.1 (1D+); no longer IC1.3 (2D+)
- net USB-C_DN: now also IC1.4 (2D-); no longer IC1.2 (1D-)
- net USB-C_DP: now also IC1.3 (2D+); no longer IC1.1 (1D+)

Commit message: PCB Routing
Parts:
- U4: renamed from IC1; Mfr. Part # (none) -> TS3USB221A-Q1; Store URL - Digikey (none) -> https://www.digikey.com/en/products/detail/texas-instrument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; Store URL - Mouser (none) -> https://eu.mouser.com/en/ProductDetail/Texas-Instruments/TS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
Changed lines of the file:
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@@
 		(in_pos_files yes)
 		(dnp no)
-		(property "Reference" "IC1"
+		(property "Reference" "U4"
 			(at 101.6 77.216 0)
 			(show_name no)
@@
 			)
 		)
-		(property "Datasheet" ""
+		(property "Datasheet" "https://www.ti.com/lit/ds/scds300e/scds300e.pdf"
 			(at 92.71 93.98 0)
 			(hide yes)
@@
 				)
 				(justify bottom)
+			)
+		)
+		(property "Mfr. Part #" "TS3USB221A-Q1 "
+			(at 92.71 93.98 0)
+			(hide yes)
+			(show_name no)
+			(do_not_autoplace no)
+			(effects
+				(font
+					(size 1.27 1.27)
+				)
+			)
+		)
+		(property "Store URL - Digikey" "https://www.digikey.com/en/products/detail/texas-instruments/TS3USB221AQRSERQ1/2356129"
+			(at 92.71 93.98 0)
+			(hide yes)
+			(show_name no)
+			(do_not_autoplace no)
+			(effects
+				(font
+					(size 1.27 1.27)
+				)
+			)
+		)
+		(property "Store URL - Mouser" "https://eu.mouser.com/en/ProductDetail/Texas-Instruments/TS3USB221AQRSERQ1?qs=0zjllh%252Bnl7aR1p0hCAkrQg%3D%3D&utm_id=24220444990&utm_source=google&utm_medium=cpc&utm_marketing_tactic=emeacorp&gad_source=1&gad_campaignid=24220444990&gbraid=0AAAAADn_wf3bBX7SFUgyO766q6os0wX-w&gclid=CjwKCAjwifjVBhBKEiwAYx4K9JuAl4mT--sc98itxdmHOnnEhai6YxXHtRtWpTKQ-h0O4Dv477LJrBoCLbMQAvD_BwE"
+			(at 92.71 93.98 0)
+			(hide yes)
+			(show_name no)
+			(do_not_autoplace no)
+			(effects
+				(font
+					(size 1.27 1.27)
+				)
 			)
 		)
@@
 			(project "MP3_Player"
 				(path "/5963f475-7f70-4482-9734-331d34890960/1923b4e2-6cf4-4620-8e30-fa635a1e0487"
-					(reference "IC1")
+					(reference "U4")
 					(unit 1)
 				)
