File: PCB/MP3_Player/MP3_Player.kicad_pcb (KiCad board)
At the start: 2 copper layers, 0 parts

Commit message: Starting PCB Layout
Parts:
- added C1: 100n, Capacitor_SMD:C_0402_1005Metric, B.Cu at (148.3, 47.9)
- added C10: 2p2, Capacitor_SMD:C_0402_1005Metric, B.Cu at (145.5, 51.9)
- added C11: 2p2, Capacitor_SMD:C_0402_1005Metric, B.Cu at (145.5, 53.8)
- added C12: 2p2, Capacitor_SMD:C_0402_1005Metric, B.Cu at (145.5, 55.8)
- added C13: 100n, Capacitor_SMD:C_0402_1005Metric, B.Cu at (59.5, 54.4)
- added C14: 1u, Capacitor_SMD:C_0402_1005Metric, B.Cu at (95.6, 153.6)
- added C15: 4u7, Capacitor_SMD:C_0603_1608Metric, B.Cu at (92.2, 153.9)
- added C16: 4u7, Capacitor_SMD:C_0603_1608Metric, B.Cu at (92.2, 156.4)
- added C17: 1u, Capacitor_SMD:C_0402_1005Metric, B.Cu at (95.6, 155.6)
- added C18: 1u, Capacitor_SMD:C_0402_1005Metric, B.Cu at (95.6, 157.6)
- added C19: 100n, Capacitor_SMD:C_0402_1005Metric, B.Cu at (95.6, 159.5)
- added C2: 100n, Capacitor_SMD:C_0402_1005Metric, B.Cu at (148.3, 49.9)
- added C20: 10n, Capacitor_SMD:C_0402_1005Metric, B.Cu at (193.4, 121.5)
- added C21: 10n, Capacitor_SMD:C_0402_1005Metric, B.Cu at (193.4, 123.5)
- added C22: 10n, Capacitor_SMD:C_0402_1005Metric, B.Cu at (193.4, 125.5)
- added C23: 10n, Capacitor_SMD:C_0402_1005Metric, B.Cu at (193.4, 127.4)
- added C24: 10n, Capacitor_SMD:C_0402_1005Metric, B.Cu at (193.4, 129.4)
- added C25: 10n, Capacitor_SMD:C_0402_1005Metric, B.Cu at (193.4, 131.4)
- added C26: 10n, Capacitor_SMD:C_0402_1005Metric, B.Cu at (193.4, 133.3)
- added C27: 1u, Capacitor_SMD:C_0402_1005Metric, B.Cu at (76.9, 122.5)
- added C28: 10u, Capacitor_SMD:C_0603_1608Metric, B.Cu at (184.4, 102.9)
- added C29: 100n, Capacitor_SMD:C_0402_1005Metric, B.Cu at (190.9, 95.8)
- added C3: 100n, Capacitor_SMD:C_0402_1005Metric, B.Cu at (148.3, 51.9)
- added C30: 100n, Capacitor_SMD:C_0402_1005Metric, B.Cu at (190.9, 97.8)
- added C31: 100n, Capacitor_SMD:C_0402_1005Metric, B.Cu at (190.9, 99.8)
- added C32: 2p2, Capacitor_SMD:C_0402_1005Metric, B.Cu at (190.9, 101.7)
- added C33: 2p2, Capacitor_SMD:C_0402_1005Metric, B.Cu at (190.9, 103.7)
- added C34: 100n, Capacitor_SMD:C_0402_1005Metric, B.Cu at (190.9, 105.7)
- added C35: 10u, Capacitor_SMD:C_0603_1608Metric, B.Cu at (133.5, 92.7)
- added C36: 100n, Capacitor_SMD:C_0402_1005Metric, B.Cu at (131.5, 94.5)
- added C37: 100n, Capacitor_SMD:C_0402_1005Metric, B.Cu at (142.6, 47.9)
- added C38: 100n, Capacitor_SMD:C_0402_1005Metric, B.Cu at (142.6, 49.9)
- added C39: 100n, Capacitor_SMD:C_0402_1005Metric, B.Cu at (221.2, 78.0)
- added C4: 100n, Capacitor_SMD:C_0402_1005Metric, B.Cu at (148.3, 53.8)
- added C40: 10u, Capacitor_Tantalum_SMD:CP_EIA-2012-15_AVX-P, B.Cu at (214.6, 78.4)
- added C41: 10u, Capacitor_Tantalum_SMD:CP_EIA-2012-15_AVX-P, B.Cu at (214.6, 81.2)
- added C42: 100n, Capacitor_SMD:C_0402_1005Metric, B.Cu at (221.2, 80.0)
- added C43: 2n2, Capacitor_SMD:C_0402_1005Metric, B.Cu at (221.2, 81.9)
- added C44: 2n2, Capacitor_SMD:C_0402_1005Metric, B.Cu at (221.2, 83.9)
- added C45: 2u2, Capacitor_SMD:C_0402_1005Metric, B.Cu at (221.2, 85.9)
- added C46: 10u, Capacitor_Tantalum_SMD:CP_EIA-2012-15_AVX-P, B.Cu at (214.6, 84.0)
- added C47: 100n, Capacitor_SMD:C_0402_1005Metric, B.Cu at (221.2, 87.8)
- added C48: 10u, Capacitor_Tantalum_SMD:CP_EIA-2012-15_AVX-P, B.Cu at (214.6, 86.8)
- added C49: 100n, Capacitor_SMD:C_0402_1005Metric, B.Cu at (218.3, 78.0)
- added C5: 10u, Capacitor_SMD:C_0603_1608Metric, B.Cu at (132.4, 38.9)
- added C50: 2u2, Capacitor_SMD:C_0402_1005Metric, B.Cu at (218.3, 80.0)
- added C51: 100n, Capacitor_SMD:C_0402_1005Metric, B.Cu at (218.3, 81.9)
- added C52: 100n, Capacitor_SMD:C_0402_1005Metric, B.Cu at (218.3, 83.9)
- added C6: 100n, Capacitor_SMD:C_0402_1005Metric, B.Cu at (148.3, 55.8)
- added C7: 1u, Capacitor_SMD:C_0402_1005Metric, B.Cu at (145.5, 47.9)
- added C8: 4u7 (LowESR < 1Ω), Capacitor_SMD:C_0603_1608Metric, B.Cu at (132.4, 41.4)
- added C9: 2p2, Capacitor_SMD:C_0402_1005Metric, B.Cu at (145.5, 49.9)
- added D1: MBR120VLSF, Diode_SMD:D_SOD-123F, B.Cu at (128.8, 121.9)
- added D2: MBR120VLSF, Diode_SMD:D_SOD-123F, B.Cu at (144.2, 121.8)
- added FB1: 600r (100MHz), Capacitor_SMD:C_0402_1005Metric, B.Cu at (142.6, 51.9)
- added FB2: 600r (100MHz), Capacitor_SMD:C_0402_1005Metric, B.Cu at (218.3, 85.9)
- added J1: TC2030, Connector:Tag-Connect_TC2030-IDC-NL_2x03_P1.27mm_Vertical, B.Cu at (117.4, 80.5)
- added J2: USB_C_Receptacle_16P, Connector_USB:USB_C_Receptacle_G-Switch_GT-USB-7010ASV, B.Cu at (152.4, 118.0)
- added J3: USB_A, Connector_USB:USB_A_CNCTech_1001-011-01101_Horizontal, B.Cu at (134.5, 133.4)
- added J5: BAT Connector, Connector_JST:JST_PH_S2B-PH-SM4-TB_1x02-1MP_P2.00mm_Horizontal, B.Cu at (121.0, 122.9)
- added J6: Micro_SD_Card, MSD-1-A:CUI_MSD-1-A, B.Cu at (121.2, 93.3)
- added J7: AudioPlugTRRS, SJ3-35044A:SAMESKY_SJ3-35044A, B.Cu at (124.6, 82.4)
- added J8: AudioPlugTRRS, SJ3-35044A:SAMESKY_SJ3-35044A, B.Cu at (144.8, 82.4)
- added JCON1: 13 Pin Flex Connector, TF29-13S-0.4SH(800):HRS_TF29-13S-0.4SH_800_, F.Cu at (350.5, 103.8)
- added JP1: Boot Select, Jumper:SolderJumper-2_P1.3mm_Bridged2Bar_RoundedPad1.0x1.5mm, B.Cu at (144.3, 99.5)
- added JP2: Boot Select, Jumper:SolderJumper-3_P1.3mm_Bridged12_RoundedPad1.0x1.5mm, B.Cu at (121.0, 49.0)
- added JP3: Addr Select, Jumper:SolderJumper-3_P1.3mm_Bridged12_RoundedPad1.0x1.5mm, B.Cu at (135.3, 52.5)
- added MK1: ICS-43434, Sensor_Audio:InvenSense_ICS-43434-6_3.5x2.65mm, F.Cu at (349.7, 137.9)
- added MK2: ICS-43434, Sensor_Audio:InvenSense_ICS-43434-6_3.5x2.65mm, F.Cu at (354.1, 137.9)
- added Q1: S8050, Package_TO_SOT_SMD:TSOT-23, B.Cu at (83.8, 127.0)
- added R1: 10k, Resistor_SMD:R_0402_1005Metric, B.Cu at (131.0, 47.9)
- added R10: 1k, Resistor_SMD:R_0402_1005Metric, B.Cu at (91.3, 149.7)
- added R11: 10r, Resistor_SMD:R_0603_1608Metric, B.Cu at (82.5, 124.0)
- added R12: 10k, Resistor_SMD:R_0402_1005Metric, B.Cu at (79.7, 125.6)
- added R13: 1k, Resistor_SMD:R_0402_1005Metric, B.Cu at (79.7, 127.5)
- added R14: 4k7, Resistor_SMD:R_0402_1005Metric, B.Cu at (131.0, 49.9)
- added R15: 4k7, Resistor_SMD:R_0402_1005Metric, B.Cu at (131.0, 51.9)
- added R16: 10k, Resistor_SMD:R_0402_1005Metric, B.Cu at (180.6, 95.8)
- added R17: 10k, Resistor_SMD:R_0402_1005Metric, B.Cu at (131.5, 91.0)
- added R18: 10k, Resistor_SMD:R_0402_1005Metric, B.Cu at (131.5, 92.1)
- added R19: 10k, Resistor_SMD:R_0402_1005Metric, B.Cu at (131.5, 98.8)
- added R2: 5k1, Resistor_SMD:R_0402_1005Metric, B.Cu at (56.4, 39.0)
- added R20: 10k, Resistor_SMD:R_0402_1005Metric, B.Cu at (131.5, 93.2)
- added R21: 10k, Resistor_SMD:R_0402_1005Metric, B.Cu at (131.5, 97.5)
- added R22: 470r, Resistor_SMD:R_0603_1608Metric, B.Cu at (201.3, 83.5)
- added R23: 470r, Resistor_SMD:R_0603_1608Metric, B.Cu at (201.3, 86.0)
- added R24: 100k, Resistor_SMD:R_0402_1005Metric, B.Cu at (197.8, 83.2)
- added R25: 10k, Resistor_SMD:R_0402_1005Metric, B.Cu at (180.6, 97.8)
- added R3: 5k1, Resistor_SMD:R_0402_1005Metric, B.Cu at (56.4, 41.0)
- added R4: 10k, Resistor_SMD:R_0402_1005Metric, B.Cu at (56.4, 43.0)
- added R5: 15k, Resistor_SMD:R_0402_1005Metric, B.Cu at (56.4, 45.0)
- added R6: 10k, Resistor_SMD:R_0402_1005Metric, B.Cu at (56.4, 47.0)
- added R7: 15k, Resistor_SMD:R_0402_1005Metric, B.Cu at (56.4, 49.0)
- added R8: 10k, Resistor_SMD:R_0402_1005Metric, B.Cu at (56.4, 51.0)
- added R9: 10k, Resistor_SMD:R_0402_1005Metric, B.Cu at (91.3, 147.7)
- added SW1: Toggle Switch, Button_Switch_SMD:SW_SPDT_CK_JS102011SAQN, B.Cu at (117.2, 108.0)
- added SW2: Push Button, Button_Switch_SMD:SW_SPST_B3U-1100P-B, F.Cu at (348.4, 112.2)
- added SW3: Push Button, Button_Switch_SMD:SW_SPST_B3U-1100P-B, F.Cu at (348.4, 117.3)
- added SW4: Push Button, Button_Switch_SMD:SW_SPST_B3U-1100P-B, F.Cu at (348.4, 122.5)
- added SW5: Push Button, Button_Switch_SMD:SW_SPST_B3U-1100P-B, F.Cu at (348.4, 127.6)
- added SW6: Push Button, Button_Switch_SMD:SW_SPST_B3U-1100P-B, F.Cu at (354.3, 112.2)
- added SW7: Push Button, Button_Switch_SMD:SW_SPST_B3U-1100P-B, F.Cu at (354.3, 117.3)
- added SW8: Push Button, Button_Switch_SMD:SW_SPST_B3U-1100P-B, F.Cu at (354.3, 122.5)
- added TP1: UART_TX, TestPoint:TestPoint_Pad_D1.0mm, B.Cu at (187.9, 96.3)
- added TP10: SDA, TestPoint:TestPoint_Pad_D1.0mm, B.Cu at (139.6, 57.6)
- added TP11: Backlight_TEST, TestPoint:TestPoint_Pad_D1.0mm, B.Cu at (76.7, 126.1)
- added TP2: UART_RX, TestPoint:TestPoint_Pad_D1.0mm, B.Cu at (187.9, 99.4)
- added TP3: BAT, TestPoint:TestPoint_Pad_D1.0mm, B.Cu at (109.7, 142.9)
- added TP4: GND, TestPoint:TestPoint_Pad_D1.0mm, B.Cu at (109.7, 145.9)
- added TP5: BQ_OUT, TestPoint:TestPoint_Pad_D1.0mm, B.Cu at (109.7, 149.0)
- added TP6: +3V3, TestPoint:TestPoint_Pad_D1.0mm, B.Cu at (109.7, 152.1)
- added TP7: HSE, TestPoint:TestPoint_Pad_D1.0mm, B.Cu at (139.6, 48.5)
- added TP8: LSE, TestPoint:TestPoint_Pad_D1.0mm, B.Cu at (139.6, 51.5)
- added TP9: SCL, TestPoint:TestPoint_Pad_D1.0mm, B.Cu at (139.6, 54.5)
- added U1: STM32F411CEU6, Package_DFN_QFN:QFN-48-1EP_7x7mm_P0.5mm_EP5.6x5.6mm, B.Cu at (140.3, 107.8)
- added U2: AP2112K-3.3, Package_TO_SOT_SMD:SOT-23-5, B.Cu at (131.0, 113.8)
- added U3: BQ24075RGTR, Package_DFN_QFN:VQFN-16-1EP_3x3mm_P0.5mm_EP1.6x1.6mm, B.Cu at (127.1, 115.8)
- added U4: TS3USB30ERSWR, Package_DFN_QFN:UQFN-10_1.4x1.8mm_P0.4mm, B.Cu at (143.1, 117.4)
- added U5: MAX17048G, MAX17048G:SON50P200X200X80-9N, B.Cu at (123.2, 113.8)
- added U6: PCM5102AQPWRQ1, Package_SO:TSSOP-20_4.4x6.5mm_P0.65mm, B.Cu at (134.5, 80.8)
- added U7: ST67W611M1A6B, ST67W611M1A6B:MODULE_ST67W611M1A6BTR, B.Cu at (146.3, 91.8)
- added U8: PCAL6408ABSHP, Package_DFN_QFN:VQFN-16-1EP_3x3mm_P0.5mm_EP1.6x1.6mm, B.Cu at (130.2, 106.2)
- added Y1: 25MHz, Crystal:Crystal_SMD_2016-4Pin_2.0x1.6mm, B.Cu at (132.4, 44.5)
- added Y2: 32.768KHz, Crystal:Crystal_SMD_2012-2Pin_2.0x1.2mm, B.Cu at (138.1, 44.5)
- added Y3: 32.768KHz, Crystal:Crystal_SMD_2012-2Pin_2.0x1.2mm, B.Cu at (184.3, 100.0)
Other:
- board outline added: 40 x 60 mm
- copper layers 2 -> 6

Commit message: PCB Layout
Parts:
- TP10, TP7, TP8, TP9: moved to F.Cu
- moved C27 271.7 mm to (346.6, 89.0)
- moved Q1 271.7 mm to (353.4, 93.5)
- moved R11 271.7 mm to (352.1, 90.5)
- moved R12 271.7 mm to (349.3, 92.1)
- moved R13 271.7 mm to (349.3, 94.1)
- moved TP11 271.7 mm to (346.3, 92.6)
- moved R24 164.8 mm to (345.0, 157.2)
- moved C20 152.2 mm to (345.3, 130.1)
- moved C21 152.2 mm to (345.3, 132.1)
- moved C22 152.2 mm to (345.3, 134.0)
- moved C23 152.2 mm to (345.3, 136.0)
- moved C24 152.2 mm to (345.3, 138.0)
- moved C25 152.2 mm to (345.3, 139.9)
- moved C26 152.2 mm to (345.3, 141.9)
- moved C52 149.7 mm to (348.5, 157.8)
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Connections:
- net Net-(JP1-A) renamed /Wireless/Boot Select
- R4 pad 2: /MCU/U_Sensing_USB-C -> /MCU/U_Sensing_USB-A
- R5 pad 1: /MCU/U_Sensing_USB-C -> /MCU/U_Sensing_USB-A
- R6 pad 2: /MCU/U_Sensing_USB-A -> /MCU/U_Sensing_USB-C
- R7 pad 1: /MCU/U_Sensing_USB-A -> /MCU/U_Sensing_USB-C

Commit message: PCB Layout
Parts:
- TP1, TP2: moved to F.Cu
- moved C13 0.76 mm to (143.8, 119.7), turned to 180 degrees
- moved R4 0.60 mm to (131.3, 120.6)
- moved R5 0.60 mm to (132.4, 120.6)
- moved TP5 0.57 mm to (134.0, 116.5)
- moved D1 0.51 mm to (129.1, 121.7)
- moved J3 0.50 mm to (135.0, 133.3)
- moved R14 0.44 mm to (129.1, 108.7)
- moved U4 0.26 mm to (143.0, 117.6), turned to 90 degrees
- moved U8 0.23 mm to (130.4, 106.0)
- moved D2 0.20 mm to (144.8, 122.8)
- moved JP1 0.10 mm to (144.3, 99.6)
- moved R15 0.10 mm to (127.0, 107.6)
- turned C31 to 180 degrees
- turned TP1 to 0 degrees
- turned TP2 to 0 degrees
Connections:
- net /USB/USB-A_DM renamed /USB/USB-A_DN
- net /USB/USB-C_DM renamed /USB/USB-C_DN
Routing:
- net /USB/+VBUS_USB-C: track 0.00 -> 7.49 mm
- net /USB/USB-C_DN: track 0.00 -> 2.73 mm
- net /USB/USB-C_DP: track 0.00 -> 2.65 mm
- net GND: vias 0 -> 7
- added copper zone on B.Cu, net /USB/+VBUS_USB-A
- added copper zone on B.Cu, net GND

Commit message: PCB Routing
Parts:
- removed U4: TS3USB30ERSWR, Package_DFN_QFN:UQFN-10_1.4x1.8mm_P0.4mm
- added IC1: TS3USB221AQRSERQ1, TS3USB221AQRSERQ1:TS3USB221AQRSERQ1, B.Cu at (140.2, 116.6)
- moved TP3 5.30 mm to (121.9, 114.1)
- moved R8 4.84 mm to (141.6, 114.5), turned to 0 degrees
- moved C13 3.98 mm to (142.1, 116.1), turned to 90 degrees
- moved R14 0.78 mm to (129.6, 109.3), turned to 90 degrees
- moved C19 0.40 mm to (121.4, 112.2)
- moved R2 0.30 mm to (146.5, 119.4)
- turned R3 to 180 degrees
Routing:
- net /Power/+VBUS: track 0.00 -> 33.8 mm
- net /Power/BAT +: track 0.00 -> 20.6 mm
- net /MCU/+VBAT: track 0.00 -> 18.6 mm
- net +3V3: track 0.00 -> 7.53 mm, vias 0 -> 14
- net /USB/+VBUS_USB-C: track 7.49 -> 13.1 mm
- net /MCU/SDA: track 0.00 -> 3.30 mm, vias 0 -> 2
- net /MCU/SCL: track 0.00 -> 2.94 mm, vias 0 -> 2
- net Net-(U3-TS): track 0.00 -> 1.86 mm
- net /USB/USB-C_CC1: track 0.00 -> 1.84 mm
- net /USB/USB-C_CC2: track 0.00 -> 1.83 mm
- net /Power/ISET: track 0.00 -> 1.66 mm
- net /MCU/U_Output SW: track 0.00 -> 1.50 mm
- net /MCU/U_Sensing_USB-A: track 0.00 -> 1.10 mm
- net /MCU/U_Sensing_USB-C: track 0.00 -> 1.10 mm
- net /MCU/ADDR_SELECT: track 0.00 -> 1.06 mm, vias 0 -> 1
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- added copper zone on B.Cu, net +3V3
- added copper zone on B.Cu, net /Power/BAT_OUT

Commit message: PCB Routing
Parts:
- moved TP10 8.46 mm to (129.2, 109.5)
- moved R8 6.71 mm to (139.4, 120.8), turned to 180 degrees
- moved TP9 6.33 mm to (131.2, 110.8)
- moved C13 3.89 mm to (139.9, 119.3), turned to -90 degrees
- moved IC1 2.85 mm to (141.8, 118.8), turned to 0 degrees
Connections:
- IC1 pad 1: /USB/USB-C_DP -> /USB/USB-A_DP
- IC1 pad 2: /USB/USB-C_DN -> /USB/USB-A_DN
- IC1 pad 3: /USB/USB-A_DP -> /USB/USB-C_DP
- IC1 pad 4: /USB/USB-A_DN -> /USB/USB-C_DN
Routing:
- net /USB/USB-A_DN: track 0.00 -> 12.7 mm
- net /MCU/U_D-: track 0.00 -> 12.4 mm, vias 0 -> 2
- net /MCU/U_D+: track 0.00 -> 12.4 mm, vias 0 -> 2
- net /MCU/SDA: track 3.30 -> 15.0 mm, vias 2 -> 3
- net /USB/USB-A_DP: track 0.00 -> 11.2 mm
- net /USB/USB-C_DP: track 2.65 -> 12.0 mm, vias 0 -> 2
- net /USB/USB-C_DN: track 2.73 -> 12.0 mm, vias 0 -> 2
- net /MCU/SCL: track 2.94 -> 10.4 mm, vias 2 -> 3
- net /MCU/VCAP: track 0.00 -> 2.80 mm
- net /MCU/SWDIO: track 0.00 -> 2.35 mm, vias 0 -> 1
- net /MCU/MUX_INT: track 0.00 -> 1.53 mm, vias 0 -> 1
- net /MCU/U_Output SW: track 1.50 -> 2.85 mm, vias 0 -> 1
- added copper zone on In2.Cu, net +3V3
- added copper zone on F.Cu, net GND
- added copper zone on In1.Cu, net GND
- added copper zone on In3.Cu, net GND
- added copper zone on In4.Cu, net GND

Commit message: PCB Routing
Parts:
- removed SW2, SW3, SW4, SW5, SW6, SW7, SW8: Push Button, Button_Switch_SMD:SW_SPST_B3U-1100P-B
- C51, C52, R24: moved to F.Cu
- moved MK2 240.5 mm to (122.0, 101.6)
- moved C52 231.1 mm to (124.7, 100.2), turned to 0 degrees
- moved R24 214.2 mm to (136.4, 108.5), turned to 0 degrees
- moved MK1 213.3 mm to (146.3, 99.3)
- moved C51 207.7 mm to (148.8, 98.0), turned to 0 degrees
- moved R12 122.3 mm to (229.6, 67.1)
- moved R13 122.3 mm to (229.6, 69.1)
- moved C27 122.3 mm to (226.9, 64.0)
- moved Q1 122.3 mm to (233.8, 68.6)
- moved R11 122.3 mm to (232.4, 65.6)
- moved TP11 122.3 mm to (226.6, 67.6)
- moved C20 122.3 mm to (225.6, 105.1)
- moved C21 122.3 mm to (225.6, 107.1)
- moved C22 122.3 mm to (225.6, 109.0)
- moved C23 122.3 mm to (225.6, 111.0)
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Routing:
- net /Audio/DAC_LRCK: track 0.00 -> 105.2 mm, vias 0 -> 2
- net /MCU/SWDIO: track 2.35 -> 78.0 mm, vias 1 -> 5
- net /Audio/MIC_WS: track 0.00 -> 62.7 mm, vias 0 -> 3
- net /MCU/SWCLK: track 0.00 -> 61.9 mm, vias 0 -> 6
- net /Audio/DAC_DIN: track 0.00 -> 61.4 mm, vias 0 -> 4
- net /MCU/SWO: track 0.00 -> 57.2 mm, vias 0 -> 2
- net +3V3: track 7.53 -> 55.1 mm, vias 14 -> 26
- net /Audio/MIC_SD: track 0.00 -> 46.1 mm, vias 0 -> 1
- net /Audio/MIC_SCK: track 0.00 -> 46.0 mm, vias 0 -> 1
- net /Audio/DAC_XSMT: track 0.00 -> 45.2 mm, vias 0 -> 2
- net /MCU/SD_CLK: track 0.00 -> 43.8 mm, vias 0 -> 4
- net /Audio/DAC_BCK: track 0.00 -> 40.9 mm, vias 0 -> 2
- net /MCU/W_Chip_EN: track 0.00 -> 38.7 mm, vias 0 -> 2
- net /MCU/NRST: track 0.00 -> 37.8 mm, vias 0 -> 4
- net GND: track 0.00 -> 36.7 mm, vias 14 -> 29
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
Commit message: PCB Routing
Parts:
- removed J7, J8: AudioPlugTRRS, SJ3-35044A:SAMESKY_SJ3-35044A
- added J4: SJ3-35044A, SJ3-35044A:SAMESKY_SJ3-35044A, B.Cu at (144.8, 82.4)
- added J9: SJ3-35044A, SJ3-35044A:SAMESKY_SJ3-35044A, B.Cu at (124.6, 82.4)
- moved C20 51.8 mm to (175.2, 117.0)
- moved C21 51.8 mm to (175.2, 119.0)
- moved C22 51.8 mm to (175.2, 120.9)
- moved C23 51.8 mm to (175.2, 122.9)
- moved C24 51.8 mm to (175.2, 124.9)
- moved C25 51.8 mm to (175.2, 126.8)
- moved C26 51.8 mm to (175.2, 128.8)
- moved C27 51.8 mm to (176.5, 75.9)
- moved Q1 51.8 mm to (183.4, 80.5)
- moved R11 51.8 mm to (182.1, 77.5)
- moved R12 51.8 mm to (179.2, 79.0)
- moved R13 51.8 mm to (179.2, 81.0)
- moved TP11 51.8 mm to (176.2, 79.5)
- moved JCON1 50.2 mm to (181.4, 87.7)
- moved TP10 4.25 mm to (133.4, 109.3)
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- renumbered IC1 to U4
Routing:
- net /Display/BL: track 2.11 -> 35.6 mm, vias 1 -> 4
- net /Audio/ROUT: track 1.34 -> 33.3 mm, vias 0 -> 2
- net /Audio/LOUT: track 1.36 -> 30.3 mm
- net /Display/CLK: track 2.68 -> 18.5 mm
- net /Display/DIN: track 2.65 -> 11.2 mm
- net /Audio/MIC_SCK: track 46.0 -> 53.7 mm
- net /Display/RST: track 2.04 -> 8.23 mm
- net /Display/CS: track 2.74 -> 8.92 mm
- net /Display/DC: track 4.33 -> 8.67 mm
- net /Audio/MIC_WS: track 62.7 -> 58.5 mm
- net /MCU/SDA: track 23.6 -> 27.1 mm
- net /MCU/ADDR_SELECT: track 1.06 -> 4.10 mm, vias 1 -> 0
- net /MCU/SCL: track 19.0 -> 21.7 mm
- net /Audio/MIC_SD: track 46.1 -> 43.9 mm
- net /MCU/W_MISO: track 28.5 -> 30.2 mm
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
Commit message: PCB Routing
Parts:
- added SW2: Push Button, Button_Switch_SMD:SW_Push_SPST_NO_Alps_SKRK, F.Cu at (129.6, 112.2)
- added SW3: Push Button, Button_Switch_SMD:SW_Push_SPST_NO_Alps_SKRK, F.Cu at (122.0, 116.8)
- added SW4: Push Button, Button_Switch_SMD:SW_Push_SPST_NO_Alps_SKRK, F.Cu at (136.1, 116.8)
- added SW5: Push Button, Button_Switch_SMD:SW_Push_SPST_NO_Alps_SKRK, F.Cu at (129.6, 121.7)
- added SW6: Push Button, Button_Switch_SMD:SW_Push_SPST_NO_Alps_SKRK, F.Cu at (129.6, 116.7)
- added SW7: Push Button, Button_Switch_SMD:SW_Push_SPST_NO_Alps_SKRK, F.Cu at (143.1, 123.0)
- added SW8: Push Button, Button_Switch_SMD:SW_Push_SPST_NO_Alps_SKRK, F.Cu at (143.1, 117.9)
- C20, C21, C22, C23, C24, C25, C26: moved to F.Cu
- moved C20 42.7 mm to (132.8, 112.0), turned to 90 degrees
- moved C21 37.5 mm to (162.8, 154.3), turned to 0 degrees
- moved C25 32.6 mm to (144.7, 115.5), turned to 0 degrees
- moved C22 31.6 mm to (162.7, 149.9), turned to 0 degrees
- moved C26 31.4 mm to (144.9, 120.7), turned to 0 degrees
- moved C23 25.8 mm to (162.7, 145.5), turned to 0 degrees
- moved C24 20.5 mm to (162.7, 141.0), turned to 0 degrees
- moved TP10 9.77 mm to (124.5, 113.1)
- moved TP9 9.16 mm to (124.4, 111.1)
- moved JCON1 0.95 mm to (180.7, 87.0)
Routing:
- net /MCU/BOOT0: track 2.17 -> 34.4 mm
- net /Buttons/V-: track 1.56 -> 25.2 mm
- net /Buttons/V+: track 0.82 -> 20.3 mm
- net /Buttons/Up: track 1.27 -> 15.5 mm
- net /MCU/SD_CLK: track 43.8 -> 54.4 mm
- net /Audio/DAC_DIN: track 61.4 -> 71.4 mm
- net GND: track 36.7 -> 41.3 mm
- net /Audio/DAC_LRCK: track 105.2 -> 109.3 mm
- net /MCU/SWCLK: track 61.9 -> 59.9 mm
- net /MCU/SCL: track 21.7 -> 20.1 mm
- net /MCU/U_Output SW: track 29.2 -> 27.6 mm
- net +3V3: track 54.9 -> 53.6 mm, vias 26 -> 27
- net /MCU/MUX_INT: track 15.7 -> 16.8 mm
- net /MCU/SWDIO: track 78.0 -> 77.0 mm, vias 5 -> 6
- net /MCU/SDA: track 27.1 -> 26.6 mm
