File: PCB/MP3_Player/MP3_Player.kicad_pcb (KiCad board)
At the start: 6 copper layers, 40 x 60 mm, 125 parts, among them J1 TC2030, J2 USB_C_Receptacle_16P, J3 USB_A, J4 SJ3-35044A, J5 BAT Connector, J6 Micro_SD_Card, J9 SJ3-35044A, Q1 S8050, SW1 Toggle Switch, SW2 Push Button, SW3 Push Button, SW4 Push Button, SW5 Push Button, SW6 Push Button, SW7 Push Button, SW8 Push Button, U1 STM32F411CEU6, U2 AP2112K-3.3, U3 BQ24075RGTR, U4 TS3USB221AQRSERQ1, U5 MAX17048G, U6 PCM5102AQPWRQ1, U7 ST67W611M1A6B, U8 PCAL6408ABSHP, Y1 25MHz, Y2 32.768KHz, Y3 32.768KHz

Commit message: PCB Routing
Parts:
- C27, Q1, R11, R12, R13, TP11: moved to F.Cu
- moved Q1 50.3 mm to (133.6, 73.6), turned to -90 degrees
- moved C21 50.0 mm to (132.7, 114.4)
- moved R13 49.3 mm to (130.4, 74.1), turned to 90 degrees
- moved R12 49.1 mm to (130.6, 72.3)
- moved R11 47.8 mm to (134.2, 76.7), turned to 0 degrees
- moved C24 44.2 mm to (125.4, 117.3), turned to -90 degrees
- moved C22 40.6 mm to (133.5, 121.7)
- moved TP11 40.4 mm to (136.2, 73.5), turned to 0 degrees
- moved C23 38.6 mm to (134.5, 119.2)
- moved C27 7.28 mm to (179.2, 82.7), turned to 0 degrees
- moved SW8 6.21 mm to (145.4, 112.2), turned to 0 degrees
- moved C25 4.51 mm to (141.1, 112.7), turned to -90 degrees
- moved C26 3.35 mm to (142.0, 122.3), turned to -90 degrees
- moved SW7 2.66 mm to (145.4, 121.8), turned to 180 degrees
- moved SW2 0.45 mm to (129.6, 111.7)
Connections:
- U8 pad 3: /Buttons/Down -> /Buttons/Left
- U8 pad 4: /Buttons/Left -> /Buttons/Down
- U8 pad 5: /Buttons/Right -> /Buttons/Ok
- U8 pad 7: /Buttons/Ok -> /Buttons/Right
Routing:
- net /Buttons/Down: track 1.14 -> 23.2 mm
- net /Buttons/Left: track 0.92 -> 18.0 mm
- net /Buttons/Right: track 0.77 -> 17.6 mm
- net /Display/CLK: track 18.5 -> 34.0 mm
- net /Display/CS: track 8.92 -> 23.6 mm
- net /Buttons/Ok: track 1.13 -> 15.4 mm
- net /Display/DIN: track 11.2 -> 24.5 mm
- net /Display/RST: track 8.23 -> 20.9 mm
- net /Display/DC: track 8.67 -> 20.8 mm
- net /Display/BL: track 35.6 -> 24.2 mm
- net /Buttons/V+: track 20.3 -> 15.2 mm
- net /Audio/MIC_SCK: track 53.6 -> 56.3 mm
- net /Buttons/V-: track 25.2 -> 23.1 mm
- net GND: track 41.3 -> 43.2 mm, vias 29 -> 28
- net /MCU/W_RDY: track 34.3 -> 35.4 mm
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
Commit message: Final PCB Routing
Parts:
- removed JCON1: 13 Pin Flex Connector, TF29-13S-0.4SH(800):HRS_TF29-13S-0.4SH_800_
- added FCON1: 26 Pins 0.5mm, Connector_FFC-FPC:Amphenol_F32R-1A7x1-11025_1x25-1MP_P0.5mm_Horizontal, F.Cu at (134.9, 91.5)
- moved C27 40.2 mm to (139.2, 86.9)
- moved TP11 7.45 mm to (132.7, 80.0)
- moved R11 1.08 mm to (133.6, 77.5), turned to -90 degrees
Connections:
- net /MCU/+VBAT renamed /Power/EN1
- net Net-(JCON1-LEDK) renamed /Display/BL_LEDK
- net Net-(U3-TS) renamed /Power/TS
- net Net-(U7-UART_RX) renamed /Wireless/UART_RX
- net Net-(U7-UART_TX) renamed /Wireless/UART_TX
- net Net-(U7-XTAL32K_IN) renamed /Wireless/XATL_IN
- net Net-(U7-XTAL32K_OUT) renamed /Wireless/XTAL_OUT
Routing:
- net /Display/BL: track 24.2 -> 53.6 mm
- net /Display/DIN: track 24.5 -> 42.0 mm, vias 1 -> 3
- net /Display/DC: track 20.8 -> 36.4 mm, vias 1 -> 3
- net /Display/RST: track 20.9 -> 34.4 mm, vias 1 -> 3
- net /Display/CS: track 23.6 -> 36.4 mm
- net /Display/CLK: track 34.0 -> 46.3 mm
- net /Display/BL_LEDK: track 0.00 -> 12.0 mm
- net +3V3: track 53.0 -> 56.8 mm
- net /Display/BL_Control: track 0.00 -> 3.05 mm
- net /Display/BL_Out: track 0.00 -> 1.73 mm
- net GND: track 43.2 -> 44.3 mm

Commit message: Routing Revision
Routing:
- net +3V3: track 56.8 -> 65.2 mm
- net /MCU/SWDIO: track 77.0 -> 78.9 mm
- net /MCU/NRST: track 37.8 -> 39.0 mm
- net GND: track 44.3 -> 43.9 mm, vias 28 -> 40

Commit message: PCB Correction
Parts:
- FCON1: footprint Connector_FFC-FPC:Amphenol_F32R-1A7x1-11025_1x25-1MP_P0.5mm_Horizontal -> Connector_FFC-FPC:Amphenol_F32R-1A7x1-11026_1x26-1MP_P0.5mm_Horizontal
- moved C51 0.22 mm to (147.2, 96.3)
- moved FCON1 0.10 mm to (135.0, 91.5)
- moved C20 0.10 mm to (132.9, 112.0)
- moved TP9 0.10 mm to (124.4, 111.0)
Routing:
- net GND: track 43.9 -> 98.1 mm, vias 40 -> 43
- net /Audio/DAC_LRCK: track 109.6 -> 101.2 mm
- net /Audio/+3V3A: track 10.8 -> 16.9 mm
- net /MCU/W_RDY: track 35.4 -> 33.0 mm
- net /MCU/SD_CLK: track 54.4 -> 53.7 mm
- net /Audio/DAC_DIN: track 71.2 -> 70.5 mm

Commit message: PCB Routing
Parts:
- moved C36 0.98 mm to (130.7, 95.0), turned to -90 degrees
Routing:
- net GND: track 98.1 -> 129.6 mm, vias 43 -> 160
- net +3V3: track 65.7 -> 74.7 mm, vias 27 -> 32
- net /Display/BL: track 53.6 -> 47.4 mm
- net /MCU/SCL: track 20.4 -> 21.6 mm, vias 4 -> 3
- net /Buttons/Up: track 15.4 -> 16.2 mm
- net /Audio/+3V3A: track 16.9 -> 17.6 mm
