File: PCB/MP3_Player/audio.kicad_sch (KiCad schematic)
At the start: 23 parts, among them J7 AudioPlug4, J8 AudioPlug4, U6 PCM5102AQPWRQ1

Commit message: Started Making BOM
Parts:
- C39, C42, C47, C49, C51, C52: Mfr. Part # (none) -> CL05B104KP5NNNC; Store URL - Digikey (none) -> https://www.digikey.pt/pt/products/detail/samsung-electro-m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; Store URL - Mouser (none) -> https://pt.mouser.com/en/ProductDetail/Samsung-Electro-Mech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
- C40, C41, C46, C48: footprint Sensor_Audio:InvenSense_ICS-43434-6_3.5x2.65mm -> (none); Mfr. Part # (none) -> T529P106M010AAE200; Store URL - Digikey (none) -> https://www.digikey.pt/pt/products/detail/kemet/T529P106M01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; Store URL - Mouser (none) -> https://pt.mouser.com/en/ProductDetail/KEMET/T529P106M010AA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
- C43, C44: Mfr. Part # (none) -> CL05B222JB5NNNC; Store URL - Digikey (none) -> https://www.digikey.pt/pt/products/detail/samsung-electro-m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; Store URL - Mouser (none) -> https://pt.mouser.com/en/ProductDetail/Samsung-Electro-Mech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
- C45, C50: Mfr. Part # (none) -> CL05A225MQ5NNND; Store URL - Digikey (none) -> https://www.digikey.pt/pt/products/detail/samsung-electro-m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; Store URL - Mouser (none) -> https://pt.mouser.com/en/ProductDetail/Samsung-Electro-Mech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

Commit message: Continue Making BOM
Parts:
- FB2: Mfr. Part # (none) -> BLM15AG601SN1D; Store URL - Digikey (none) -> https://www.digikey.pt/pt/products/detail/murata-electronic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; Store URL - Mouser (none) -> https://pt.mouser.com/en/ProductDetail/Murata-Electronics/B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
- MK1, MK2: Mfr. Part # (none) -> ICS-43434; Store URL - Digikey (none) -> https://www.digikey.pt/pt/products/detail/tdk-invensense/IC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; Store URL - Mouser (none) -> https://pt.mouser.com/en/ProductDetail/TDK-InvenSense/ICS-4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
- R22, R23: Mfr. Part # (none) -> CRCW0603470RFKEA; Store URL - Digikey (none) -> https://www.digikey.pt/pt/products/detail/vishay-dale/CRCW0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; Store URL - Mouser (none) -> https://pt.mouser.com/en/ProductDetail/Vishay/CRCW0603470RF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
- R24: Mfr. Part # (none) -> CRCW0402100KFKED; Store URL - Digikey (none) -> https://www.digikey.pt/pt/products/detail/vishay-dale/CRCW0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; Store URL - Mouser (none) -> https://pt.mouser.com/en/ProductDetail/Vishay/CRCW0402100KF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
Changed lines of the file:
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@@
 			)
 		)
-		(property "Datasheet" ""
+		(property "Datasheet" "https://www.vishay.com/docs/20035/dcrcwe3.pdf"
 			(at 95.25 161.29 0)
 			(hide yes)
@@
 			)
 		)
-		(property "Description" "Resistor"
+		(property "Description" "0402"
 			(at 95.25 161.29 0)
 			(hide yes)
@@
 		)
 		(property "Store URL - TME" ""
+			(at 95.25 161.29 0)
+			(hide yes)
+			(show_name no)
+			(do_not_autoplace no)
+			(effects
+				(font
+					(size 1.27 1.27)
+				)
+			)
+		)
+		(property "Mfr. Part #" "CRCW0402100KFKED"
+			(at 95.25 161.29 0)
+			(hide yes)
+			(show_name no)
+			(do_not_autoplace no)
+			(effects
+				(font
+					(size 1.27 1.27)
+				)
+			)
+		)
+		(property "Store URL - Digikey" "https://www.digikey.pt/pt/products/detail/vishay-dale/CRCW0402100KFKED/1178235"
+			(at 95.25 161.29 0)
+			(hide yes)
+			(show_name no)
+			(do_not_autoplace no)
+			(effects
+				(font
+					(size 1.27 1.27)
+				)
+			)
+		)
+		(property "Store URL - Mouser" "https://pt.mouser.com/en/ProductDetail/Vishay/CRCW0402100KFKED?qs=OlqPY1CiralZGKRwQ4Glcg%3D%3D"
 			(at 95.25 161.29 0)
 			(hide yes)
@@
 			)
 		)
+		(property "Mfr. Part #" "ICS-43434"
+			(at 73.66 105.41 0)
+			(hide yes)
+			(show_name no)
+			(do_not_autoplace no)
+			(effects
+				(font
+					(size 1.27 1.27)
+				)
+			)
+		)
+		(property "Store URL - Digikey" "https://www.digikey.pt/pt/products/detail/tdk-invensense/ICS-43434/6140298"
+			(at 73.66 105.41 0)
+			(hide yes)
+			(show_name no)
+			(do_not_autoplace no)
+			(effects
+				(font
+					(size 1.27 1.27)
+				)
+			)
+		)
+		(property "Store URL - Mouser" "https://pt.mouser.com/en/ProductDetail/TDK-InvenSense/ICS-43434?qs=u4fy%2FsgLU9PAgmWRI7%252BqXA%3D%3D"
+			(at 73.66 105.41 0)
+			(hide yes)
+			(show_name no)
+			(do_not_autoplace no)
+			(effects
+				(font
+					(size 1.27 1.27)
+				)
+			)
+		)
 		(pin "6"
 		)
@@
 			)
 		)
-		(property "Datasheet" ""
+		(property "Datasheet" "https://pim.murata.com/asset/pim4/ferriteBeadInductortypefilter/ENFA0018_PDF_FERRITEBEADINDUCTORTYPEFILTER?lastModifiedDatetime=20250707191428"
 			(at 151.13 48.26 0)
 			(hide yes)
@@
 			)
 		)
-		(property "Description" "Ferrite bead"
+		(property "Description" "0402"
 			(at 151.13 48.26 0)
 			(hide yes)
@@
 		)
 		(property "Store URL - TME" ""
+			(at 151.13 48.26 90)
+			(hide yes)
+			(show_name no)
+			(do_not_autoplace no)
+			(effects
+				(font
+					(size 1.27 1.27)
+				)
+			)
+		)
+		(property "Mfr. Part #" "BLM15AG601SN1D"
+			(at 151.13 48.26 90)
+			(hide yes)
+			(show_name no)
+			(do_not_autoplace no)
+			(effects
+				(font
+					(size 1.27 1.27)
+				)
+			)
+		)
+		(property "Store URL - Digikey" "https://www.digikey.pt/pt/products/detail/murata-electronics/BLM15AG601SN1D/584217"
+			(at 151.13 48.26 90)
+			(hide yes)
+			(show_name no)
+			(do_not_autoplace no)
+			(effects
+				(font
+					(size 1.27 1.27)
+				)
+			)
+		)
+		(property "Store URL - Mouser" "https://pt.mouser.com/en/ProductDetail/Murata-Electronics/BLM15AG601SN1D?qs=%2FjCH2pcB5WLSIF5DG9Nbqw%3D%3D"
 			(at 151.13 48.26 90)
 			(hide yes)
@@
 			)
 		)
-		(property "Datasheet" ""
+		(property "Datasheet" "https://www.vishay.com/docs/20035/dcrcwe3.pdf"
 			(at 172.72 82.55 0)
 			(hide yes)
@@
 			)
 		)
-		(property "Description" "Resistor"
+		(property "Description" "0603"
 			(at 172.72 82.55 0)
 			(hide yes)
@@
 		)
 		(property "Store URL - TME" ""
+			(at 172.72 82.55 90)
+			(hide yes)
+			(show_name no)
+			(do_not_autoplace no)
+			(effects
+				(font
+					(size 1.27 1.27)
+				)
+			)
+		)
+		(property "Mfr. Part #" "CRCW0603470RFKEA"
+			(at 172.72 82.55 90)
+			(hide yes)
+			(show_name no)
+			(do_not_autoplace no)
+			(effects
+				(font
+					(size 1.27 1.27)
+				)
+			)
+		)
+		(property "Store URL - Digikey" "https://www.digikey.pt/pt/products/detail/vishay-dale/CRCW0603470RFKEA/1174630"
+			(at 172.72 82.55 90)
+			(hide yes)
+			(show_name no)
+			(do_not_autoplace no)
+			(effects
+				(font
+					(size 1.27 1.27)
+				)
+			)
+		)
+		(property "Store URL - Mouser" "https://pt.mouser.com/en/ProductDetail/Vishay/CRCW0603470RFKEA?qs=2LLIXXYaQepTa3IToKeExA%3D%3D"
 			(at 172.72 82.55 90)
 			(hide yes)
@@
 			)
 		)
-		(property "Datasheet" ""
+		(property "Datasheet" "https://www.vishay.com/docs/20035/dcrcwe3.pdf"
 			(at 172.72 80.01 0)
 			(hide yes)
@@
 			)
 		)
-		(property "Description" "Resistor"
+		(property "Description" "0603"
 			(at 172.72 80.01 0)
 			(hide yes)
@@
 		)
 		(property "Store URL - TME" ""
+			(at 172.72 80.01 90)
+			(hide yes)
+			(show_name no)
+			(do_not_autoplace no)
+			(effects
+				(font
+					(size 1.27 1.27)
+				)
+			)
+		)
+		(property "Mfr. Part #" "CRCW0603470RFKEA"
+			(at 172.72 80.01 90)
+			(hide yes)
+			(show_name no)
+			(do_not_autoplace no)
+			(effects
+				(font
+					(size 1.27 1.27)
+				)
+			)
+		)
+		(property "Store URL - Digikey" "https://www.digikey.pt/pt/products/detail/vishay-dale/CRCW0603470RFKEA/1174630"
+			(at 172.72 80.01 90)
+			(hide yes)
+			(show_name no)
+			(do_not_autoplace no)
+			(effects
+				(font
+					(size 1.27 1.27)
+				)
+			)
+		)
+		(property "Store URL - Mouser" "https://pt.mouser.com/en/ProductDetail/Vishay/CRCW0603470RFKEA?qs=2LLIXXYaQepTa3IToKeExA%3D%3D"
 			(at 172.72 80.01 90)
 			(hide yes)
@@
 			(at 73.66 153.67 0)
 			(hide yes)
+			(show_name no)
+			(do_not_autoplace no)
+			(effects
+				(font
+					(size 1.27 1.27)
+				)
+			)
+		)
+		(property "Mfr. Part #" "ICS-43434"
+			(at 73.66 153.67 0)
+			(hide yes)
+			(show_name no)
+			(do_not_autoplace no)
+			(effects
+				(font
+					(size 1.27 1.27)
+				)
+			)
+		)
+		(property "Store URL - Digikey" "https://www.digikey.pt/pt/products/detail/tdk-invensense/ICS-43434/6140298"
+			(at 73.66 153.67 0)
+			(hide yes)
+			(show_name no)
+			(do_not_autoplace no)
+			(effects
+				(font
+					(size 1.27 1.27)
+				)
+			)
+		)
+		(property "Store URL - Mouser" "https://pt.mouser.com/en/ProductDetail/TDK-InvenSense/ICS-43434?qs=u4fy%2FsgLU9PAgmWRI7%252BqXA%3D%3D"
+			(at 73.66 153.67 0)
+			(hide yes)

Commit message: Finished BOM; Started Footprint assignment
Parts:
- C39, C42, C43, C44, C45, C47, C49, C50, C51, C52, FB2, R24: footprint (none) -> Capacitor_SMD:C_0402_1005Metric
- C40, C41, C46, C48: footprint (none) -> Capacitor_Tantalum_SMD:CP_EIA-2012-15_AVX-P
- J7, J8: Mfr. Part # (none) -> ASJ-190-A; Store URL - Digikey (none) -> https://www.digikey.pt/pt/products/detail/adam-tech/ASJ-190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; Store URL - Mouser (none) -> https://pt.mouser.com/en/ProductDetail/Adam-Tech/ASJ-190-A?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
- R22, R23: footprint (none) -> Capacitor_SMD:C_0603_1608Metric
Changed lines of the file:
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@@
 			)
 		)
-		(property "Footprint" ""
+		(property "Footprint" "Capacitor_SMD:C_0402_1005Metric"
 			(at 93.472 161.29 90)
 			(hide yes)
@@
 			)
 		)
-		(property "Datasheet" ""
+		(property "Datasheet" "https://app.adam-tech.com/products/download/data_sheet/203691/asj-190-x-data-sheet.pdf"
 			(at 223.52 52.07 0)
 			(hide yes)
@@
 			)
 		)
+		(property "Mfr. Part #" "ASJ-190-A"
+			(at 232.41 54.61 0)
+			(hide yes)
+			(show_name no)
+			(do_not_autoplace no)
+			(effects
+				(font
+					(size 1.27 1.27)
+				)
+			)
+		)
+		(property "Store URL - Digikey" "https://www.digikey.pt/pt/products/detail/adam-tech/ASJ-190-A/9831581"
+			(at 232.41 54.61 0)
+			(hide yes)
+			(show_name no)
+			(do_not_autoplace no)
+			(effects
+				(font
+					(size 1.27 1.27)
+				)
+			)
+		)
+		(property "Store URL - Mouser" "https://pt.mouser.com/en/ProductDetail/Adam-Tech/ASJ-190-A?qs=HoCaDK9Nz5dToh9HC6AKDA%3D%3D"
+			(at 232.41 54.61 0)
+			(hide yes)
+			(show_name no)
+			(do_not_autoplace no)
+			(effects
+				(font
+					(size 1.27 1.27)
+				)
+			)
+		)
 		(pin "R2"
 		)
@@
 			)
 		)
-		(property "Footprint" ""
+		(property "Footprint" "Capacitor_SMD:C_0402_1005Metric"
 			(at 192.7352 80.01 0)
 			(hide yes)
@@
 			)
 		)
-		(property "Footprint" ""
+		(property "Footprint" "Capacitor_SMD:C_0402_1005Metric"
 			(at 151.13 50.038 90)
 			(hide yes)
@@
 			)
 		)
-		(property "Footprint" ""
+		(property "Footprint" "Capacitor_SMD:C_0402_1005Metric"
 			(at 173.6852 57.15 0)
 			(hide yes)
@@
 			)
 		)
-		(property "Footprint" ""
+		(property "Footprint" "Capacitor_SMD:C_0402_1005Metric"
 			(at 204.1652 110.49 0)
 			(hide yes)
@@
 			)
 		)
-		(property "Footprint" ""
+		(property "Footprint" "Capacitor_SMD:C_0402_1005Metric"
 			(at 171.1452 95.25 0)
 			(hide yes)
@@
 			)
 		)
-		(property "Footprint" ""
+		(property "Footprint" "Capacitor_Tantalum_SMD:CP_EIA-2012-15_AVX-P"
 			(at 115.2652 58.42 0)
 			(hide yes)
@@
 			)
 		)
-		(property "Footprint" ""
+		(property "Footprint" "Capacitor_SMD:C_0402_1005Metric"
 			(at 127.9652 58.42 0)
 			(hide yes)
@@
 			)
 		)
-		(property "Footprint" ""
+		(property "Footprint" "Capacitor_SMD:C_0603_1608Metric"
 			(at 172.72 80.772 90)
 			(hide yes)
@@
 			)
 		)
-		(property "Footprint" ""
+		(property "Footprint" "Capacitor_Tantalum_SMD:CP_EIA-2012-15_AVX-P"
 			(at 192.7352 110.49 0)
 			(hide yes)
@@
 			)
 		)
-		(property "Footprint" ""
+		(property "Footprint" "Capacitor_SMD:C_0402_1005Metric"
 			(at 57.4548 99.06 0)
 			(hide yes)
@@
 			)
 		)
-		(property "Footprint" ""
+		(property "Footprint" "Capacitor_SMD:C_0402_1005Metric"
 			(at 169.8752 111.76 0)
 			(hide yes)
@@
 			)
 		)
-		(property "Footprint" ""
+		(property "Footprint" "Capacitor_SMD:C_0402_1005Metric"
 			(at 57.4548 147.32 0)
 			(hide yes)
@@
 			)
 		)
-		(property "Footprint" ""
+		(property "Footprint" "Capacitor_SMD:C_0603_1608Metric"
 			(at 172.72 81.788 90)
 			(hide yes)
@@
 			)
 		)
-		(property "Footprint" ""
+		(property "Footprint" "Capacitor_Tantalum_SMD:CP_EIA-2012-15_AVX-P"
 			(at 160.9852 57.15 0)
 			(hide yes)
@@
 			)
 		)
-		(property "Datasheet" ""
+		(property "Datasheet" "https://app.adam-tech.com/products/download/data_sheet/203691/asj-190-x-data-sheet.pdf"
 			(at 223.52 69.85 0)
 			(hide yes)
@@
 			)
 		)
+		(property "Mfr. Part #" "ASJ-190-A"
+			(at 232.41 72.39 0)
+			(hide yes)
+			(show_name no)
+			(do_not_autoplace no)
+			(effects
+				(font
+					(size 1.27 1.27)
+				)
+			)
+		)
+		(property "Store URL - Digikey" "https://www.digikey.pt/pt/products/detail/adam-tech/ASJ-190-A/9831581"
+			(at 232.41 72.39 0)
+			(hide yes)
+			(show_name no)
+			(do_not_autoplace no)
+			(effects
+				(font
+					(size 1.27 1.27)
+				)
+			)
+		)
+		(property "Store URL - Mouser" "https://pt.mouser.com/en/ProductDetail/Adam-Tech/ASJ-190-A?qs=HoCaDK9Nz5dToh9HC6AKDA%3D%3D"
+			(at 232.41 72.39 0)
+			(hide yes)
+			(show_name no)
+			(do_not_autoplace no)
+			(effects
+				(font
+					(size 1.27 1.27)
+				)
+			)
+		)
 		(pin "R2"
 		)
@@
 			)
 		)
-		(property "Footprint" ""
+		(property "Footprint" "Capacitor_SMD:C_0402_1005Metric"
 			(at 204.1652 80.01 0)
 			(hide yes)
@@
 			)
 		)
-		(property "Footprint" ""
+		(property "Footprint" "Capacitor_Tantalum_SMD:CP_EIA-2012-15_AVX-P"
 			(at 133.0452 72.39 0)
 			(hide yes)
@@
 			)
 		)
-		(property "Footprint" ""
+		(property "Footprint" "Capacitor_SMD:C_0402_1005Metric"
 			(at 143.2052 72.39 0)
 			(hide yes)

Commit message: Footprint Assingment
Parts:
- J7, J8: value AudioPlug4 -> AudioPlugTRRS; footprint Package_TO_SOT_SMD:SOT-323_SC-70 -> (none); Mfr. Part # ASJ-190-A -> ASJ-147B-R-G-KT-T/R; Store URL - Digikey https://www.digikey.pt/pt/products/detail/adam-tech/ASJ-190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 -> https://www.digikey.pt/pt/products/detail/adam-tech/ASJ-147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; Store URL - Mouser https://pt.mouser.com/en/ProductDetail/Adam-Tech/ASJ-190-A?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 -> https://pt.mouser.com/en/ProductDetail/Adam-Tech/ASJ-147B-R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
- R22, R23: footprint Capacitor_SMD:C_0603_1608Metric -> Resistor_SMD:R_0603_1608Metric
- R24: footprint Capacitor_SMD:C_0402_1005Metric -> Resistor_SMD:R_0402_1005Metric
Changed lines of the file:
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@@
 			)
 		)
-		(property "Footprint" "Capacitor_SMD:C_0402_1005Metric"
+		(property "Footprint" "Resistor_SMD:R_0402_1005Metric"
 			(at 93.472 161.29 90)
 			(hide yes)
@@
 			)
 		)
-		(property "Value" "AudioPlug4"
+		(property "Value" "AudioPlugTRRS"
 			(at 232.41 60.96 0)
 			(show_name no)
@@
 			)
 		)
-		(property "Footprint" "Package_TO_SOT_SMD:SOT-323_SC-70"
+		(property "Footprint" ""
 			(at 223.52 52.07 0)
 			(hide yes)
@@
 			)
 		)
-		(property "Datasheet" "https://app.adam-tech.com/products/download/data_sheet/203691/asj-190-x-data-sheet.pdf"
+		(property "Datasheet" "https://app.adam-tech.com/resources/download/65/ecatalog-2026.pdf"
 			(at 223.52 52.07 0)
 			(hide yes)
@@
 			)
 		)
-		(property "Mfr. Part #" "ASJ-190-A"
+		(property "Mfr. Part #" "ASJ-147B-R-G-KT-T/R"
 			(at 232.41 54.61 0)
 			(hide yes)
@@
 			)
 		)
-		(property "Store URL - Digikey" "https://www.digikey.pt/pt/products/detail/adam-tech/ASJ-190-A/9831581"
+		(property "Store URL - Digikey" "https://www.digikey.pt/pt/products/detail/adam-tech/ASJ-147B-R-G-KT-T-R/26685636"
 			(at 232.41 54.61 0)
 			(hide yes)
@@
 			)
 		)
-		(property "Store URL - Mouser" "https://pt.mouser.com/en/ProductDetail/Adam-Tech/ASJ-190-A?qs=HoCaDK9Nz5dToh9HC6AKDA%3D%3D"
+		(property "Store URL - Mouser" "https://pt.mouser.com/en/ProductDetail/Adam-Tech/ASJ-147B-R-G-KT-T-R?qs=ST9lo4GX8V2ZS4l71VM71A%3D%3D"
 			(at 232.41 54.61 0)
 			(hide yes)
@@
 			)
 		)
-		(property "Footprint" "Capacitor_SMD:C_0603_1608Metric"
+		(property "Footprint" "Resistor_SMD:R_0603_1608Metric"
 			(at 172.72 80.772 90)
 			(hide yes)
@@
 			)
 		)
-		(property "Footprint" "Capacitor_SMD:C_0603_1608Metric"
+		(property "Footprint" "Resistor_SMD:R_0603_1608Metric"
 			(at 172.72 81.788 90)
 			(hide yes)
@@
 			)
 		)
-		(property "Value" "AudioPlug4"
+		(property "Value" "AudioPlugTRRS"
 			(at 232.41 78.74 0)
 			(show_name no)
@@
 			)
 		)
-		(property "Footprint" "Package_TO_SOT_SMD:SOT-323_SC-70"
+		(property "Footprint" ""
 			(at 223.52 69.85 0)
 			(hide yes)
@@
 			)
 		)
-		(property "Datasheet" "https://app.adam-tech.com/products/download/data_sheet/203691/asj-190-x-data-sheet.pdf"
+		(property "Datasheet" "https://app.adam-tech.com/resources/download/65/ecatalog-2026.pdf"
 			(at 223.52 69.85 0)
 			(hide yes)
@@
 			)
 		)
-		(property "Mfr. Part #" "ASJ-190-A"
+		(property "Mfr. Part #" "ASJ-147B-R-G-KT-T/R"
 			(at 232.41 72.39 0)
 			(hide yes)
@@
 			)
 		)
-		(property "Store URL - Digikey" "https://www.digikey.pt/pt/products/detail/adam-tech/ASJ-190-A/9831581"
+		(property "Store URL - Digikey" "https://www.digikey.pt/pt/products/detail/adam-tech/ASJ-147B-R-G-KT-T-R/26685636"
 			(at 232.41 72.39 0)
 			(hide yes)
@@
 			)
 		)
-		(property "Store URL - Mouser" "https://pt.mouser.com/en/ProductDetail/Adam-Tech/ASJ-190-A?qs=HoCaDK9Nz5dToh9HC6AKDA%3D%3D"
+		(property "Store URL - Mouser" "https://pt.mouser.com/en/ProductDetail/Adam-Tech/ASJ-147B-R-G-KT-T-R?qs=ST9lo4GX8V2ZS4l71VM71A%3D%3D"
 			(at 232.41 72.39 0)
 			(hide yes)

Commit message: Footprint Assingment Complete
Parts:
- J7, J8: footprint (none) -> SJ3-35044A:SAMESKY_SJ3-35044A; Mfr. Part # ASJ-147B-R-G-KT-T/R -> SJ3-35044A; Store URL - Digikey https://www.digikey.pt/pt/products/detail/adam-tech/ASJ-147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 -> https://www.digikey.pt/pt/products/detail/same-sky-formerly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; Store URL - Mouser https://pt.mouser.com/en/ProductDetail/Adam-Tech/ASJ-147B-R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 -> https://pt.mouser.com/en/ProductDetail/Same-Sky/SJ3-35044A?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
Changed lines of the file:
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@@
 			)
 		)
-		(property "Footprint" ""
+		(property "Footprint" "SJ3-35044A:SAMESKY_SJ3-35044A"
 			(at 223.52 52.07 0)
 			(hide yes)
@@
 			)
 		)
-		(property "Datasheet" "https://app.adam-tech.com/resources/download/65/ecatalog-2026.pdf"
+		(property "Datasheet" "https://www.cuidevices.com/product/resource/digikeypdf/sj3-35044a.pdf"
 			(at 223.52 52.07 0)
 			(hide yes)
@@
 			)
 		)
-		(property "Mfr. Part #" "ASJ-147B-R-G-KT-T/R"
+		(property "Mfr. Part #" "SJ3-35044A"
 			(at 232.41 54.61 0)
 			(hide yes)
@@
 			)
 		)
-		(property "Store URL - Digikey" "https://www.digikey.pt/pt/products/detail/adam-tech/ASJ-147B-R-G-KT-T-R/26685636"
+		(property "Store URL - Digikey" "https://www.digikey.pt/pt/products/detail/same-sky-formerly-cui-devices/SJ3-35044A/24627965"
 			(at 232.41 54.61 0)
 			(hide yes)
@@
 			)
 		)
-		(property "Store URL - Mouser" "https://pt.mouser.com/en/ProductDetail/Adam-Tech/ASJ-147B-R-G-KT-T-R?qs=ST9lo4GX8V2ZS4l71VM71A%3D%3D"
+		(property "Store URL - Mouser" "https://pt.mouser.com/en/ProductDetail/Same-Sky/SJ3-35044A?qs=IKkN%2F947nfA%2F9r2%2FyF4SEA%3D%3D"
 			(at 232.41 54.61 0)
 			(hide yes)
@@
 			)
 		)
-		(property "Footprint" ""
+		(property "Footprint" "SJ3-35044A:SAMESKY_SJ3-35044A"
 			(at 223.52 69.85 0)
 			(hide yes)
@@
 			)
 		)
-		(property "Datasheet" "https://app.adam-tech.com/resources/download/65/ecatalog-2026.pdf"
+		(property "Datasheet" "https://www.cuidevices.com/product/resource/digikeypdf/sj3-35044a.pdf"
 			(at 223.52 69.85 0)
 			(hide yes)
@@
 			)
 		)
-		(property "Mfr. Part #" "ASJ-147B-R-G-KT-T/R"
+		(property "Mfr. Part #" "SJ3-35044A"
 			(at 232.41 72.39 0)
 			(hide yes)
@@
 			)
 		)
-		(property "Store URL - Digikey" "https://www.digikey.pt/pt/products/detail/adam-tech/ASJ-147B-R-G-KT-T-R/26685636"
+		(property "Store URL - Digikey" "https://www.digikey.pt/pt/products/detail/same-sky-formerly-cui-devices/SJ3-35044A/24627965"
 			(at 232.41 72.39 0)
 			(hide yes)
@@
 			)
 		)
-		(property "Store URL - Mouser" "https://pt.mouser.com/en/ProductDetail/Adam-Tech/ASJ-147B-R-G-KT-T-R?qs=ST9lo4GX8V2ZS4l71VM71A%3D%3D"
+		(property "Store URL - Mouser" "https://pt.mouser.com/en/ProductDetail/Same-Sky/SJ3-35044A?qs=IKkN%2F947nfA%2F9r2%2FyF4SEA%3D%3D"
 			(at 232.41 72.39 0)
 			(hide yes)

Commit message: Starting PCB Layout
Connections:
- net LDO_OUT: now reaches C41.1, C42.1, U6.18 (LDOO)
- net VNEG_CAP: now reaches C50.1, U6.5 (VNEG)
Changed lines of the file:
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@@
+		)
+	)
+	(label "LDO_OUT"
+		(at 180.34 100.33 0)
+		(effects
+			(font
+				(size 1.27 1.27)
+			)
+			(justify left bottom)
 		)
 	)
@@
 			)
 			(justify left bottom)
+		)
+	)
+	(label "VNEG_CAP"
+		(at 168.91 102.87 0)
+		(effects
+			(font
+				(size 1.27 1.27)
+			)
+			(justify left bottom)

Commit message: PCB Routing
Parts:
- removed J7, J8: AudioPlugTRRS, SJ3-35044A:SAMESKY_SJ3-35044A, symbol Connector_Audio:AudioPlug4
- added J4, J9: SJ3-35044A, SJ3-35044A:SAMESKY_SJ3-35044A, symbol SJ3-35044A:SJ3-35044A
Connections:
- net GND: now also J4.3 (R2), J9.3 (R2)
- net LOUT: now also J4.2_1 (T), J4.2_2, J9.2_1 (T), J9.2_2
- net ROUT: now also J4.4 (R1), J9.4 (R1)

Commit message: PCB Routing
Parts:
- J4, J9: Mfr. Part # (none) -> SJ3-35044A; Store URL - Digikey (none) -> https://www.digikey.pt/pt/products/detail/same-sky-formerly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
Changed lines of the file:
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@@
 			)
 		)
-		(property "Datasheet" ""
+		(property "Datasheet" "https://www.sameskydevices.com/product/resource/sj3-35044a.pdf"
 			(at 229.87 71.12 0)
 			(hide yes)
@@
 				)
 				(justify bottom)
+			)
+		)
+		(property "Mfr. Part #" "SJ3-35044A"
+			(at 229.87 71.12 0)
+			(hide yes)
+			(show_name no)
+			(do_not_autoplace no)
+			(effects
+				(font
+					(size 1.27 1.27)
+				)
+			)
+		)
+		(property "Store URL - Digikey" "https://www.digikey.pt/pt/products/detail/same-sky-formerly-cui-devices/SJ3-35044A/24627965?s=N4IgTCBcDaIMoCkDMBaJBWADAFmwQRAF0BfIA"
+			(at 229.87 71.12 0)
+			(hide yes)
+			(show_name no)
+			(do_not_autoplace no)
+			(effects
+				(font
+					(size 1.27 1.27)
+				)
 			)
 		)
@@
 			)
 		)
-		(property "Datasheet" ""
+		(property "Datasheet" "https://www.sameskydevices.com/product/resource/sj3-35044a.pdf"
 			(at 229.87 53.34 0)
 			(hide yes)
@@
 			)
 		)
+		(property "Mfr. Part #" "SJ3-35044A"
+			(at 229.87 53.34 0)
+			(hide yes)
+			(show_name no)
+			(do_not_autoplace no)
+			(effects
+				(font
+					(size 1.27 1.27)
+				)
+			)
+		)
+		(property "Store URL - Digikey" "https://www.digikey.pt/pt/products/detail/same-sky-formerly-cui-devices/SJ3-35044A/24627965?s=N4IgTCBcDaIMoCkDMBaJBWADAFmwQRAF0BfIA"
+			(at 229.87 53.34 0)
+			(hide yes)
+			(show_name no)
+			(do_not_autoplace no)
+			(effects
+				(font
+					(size 1.27 1.27)
+				)
+			)
+		)
