File: PCB/MP3_Player/buttons.kicad_sch (KiCad schematic)
At the start: 14 parts, among them SW2 Up, SW3 Left, SW4 Right, SW5 Down, SW6 OK, SW7 Volume -, SW8 Volume +

Commit message: Started Making BOM
Parts:
- C20, C21, C22, C23, C24, C25, C26: Mfr. Part # (none) -> CL05B103KB5NNND; Store URL - Digikey (none) -> https://www.digikey.pt/pt/products/detail/samsung-electro-m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; Store URL - Mouser (none) -> https://pt.mouser.com/en/ProductDetail/Samsung-Electro-Mech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

Commit message: Continue Making BOM
Parts:
- SW2: value Up -> Push Button; Mfr. Part # (none) -> B3U-1100PM-B; Store URL - Digikey (none) -> https://www.digikey.pt/pt/products/detail/aratas-formerly-o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; Store URL - Mouser (none) -> https://pt.mouser.com/en/ProductDetail/Omron-Electronics/B3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
- SW3: value Left -> Push Button; Mfr. Part # (none) -> B3U-1100PM-B; Store URL - Digikey (none) -> https://www.digikey.pt/pt/products/detail/aratas-formerly-o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; Store URL - Mouser (none) -> https://pt.mouser.com/en/ProductDetail/Omron-Electronics/B3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
- SW4: value Right -> Push Button; Mfr. Part # (none) -> B3U-1100PM-B; Store URL - Digikey (none) -> https://www.digikey.pt/pt/products/detail/aratas-formerly-o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; Store URL - Mouser (none) -> https://pt.mouser.com/en/ProductDetail/Omron-Electronics/B3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
- SW5: value Down -> Push Button; Mfr. Part # (none) -> B3U-1100PM-B; Store URL - Digikey (none) -> https://www.digikey.pt/pt/products/detail/aratas-formerly-o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; Store URL - Mouser (none) -> https://pt.mouser.com/en/ProductDetail/Omron-Electronics/B3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
- SW6: value OK -> Push Button; Mfr. Part # (none) -> B3U-1100PM-B; Store URL - Digikey (none) -> https://www.digikey.pt/pt/products/detail/aratas-formerly-o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; Store URL - Mouser (none) -> https://pt.mouser.com/en/ProductDetail/Omron-Electronics/B3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
- SW7: value Volume - -> Push Button; Mfr. Part # (none) -> B3U-1100PM-B; Store URL - Digikey (none) -> https://www.digikey.pt/pt/products/detail/aratas-formerly-o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; Store URL - Mouser (none) -> https://pt.mouser.com/en/ProductDetail/Omron-Electronics/B3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
- SW8: value Volume + -> Push Button; Mfr. Part # (none) -> B3U-1100PM-B; Store URL - Digikey (none) -> https://www.digikey.pt/pt/products/detail/aratas-formerly-o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; Store URL - Mouser (none) -> https://pt.mouser.com/en/ProductDetail/Omron-Electronics/B3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
Other:
- note added: "Down"
- note added: "Left"
- note added: "OK"
- note added: "Right"
- note added: "UP"
- note added: "V-"

Commit message: Finished BOM; Started Footprint assignment
Parts:
- C20, C21, C22, C23, C24, C25, C26: footprint (none) -> Capacitor_SMD:C_0402_1005Metric
Changed lines of the file:
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@@
 			)
 		)
-		(property "Footprint" ""
+		(property "Footprint" "Capacitor_SMD:C_0402_1005Metric"
 			(at 199.0852 119.38 0)
 			(hide yes)
@@
 			)
 		)
-		(property "Footprint" ""
+		(property "Footprint" "Capacitor_SMD:C_0402_1005Metric"
 			(at 97.4852 81.28 0)
 			(hide yes)
@@
 			)
 		)
-		(property "Footprint" ""
+		(property "Footprint" "Capacitor_SMD:C_0402_1005Metric"
 			(at 169.8752 99.06 0)
 			(hide yes)
@@
 			)
 		)
-		(property "Footprint" ""
+		(property "Footprint" "Capacitor_SMD:C_0402_1005Metric"
 			(at 199.0852 78.74 0)
 			(hide yes)
@@
 			)
 		)
-		(property "Footprint" ""
+		(property "Footprint" "Capacitor_SMD:C_0402_1005Metric"
 			(at 68.2752 81.28 0)
 			(hide yes)
@@
 			)
 		)
-		(property "Footprint" ""
+		(property "Footprint" "Capacitor_SMD:C_0402_1005Metric"
 			(at 199.0852 99.06 0)
 			(hide yes)
@@
 			)
 		)
-		(property "Footprint" ""
+		(property "Footprint" "Capacitor_SMD:C_0402_1005Metric"
 			(at 228.2952 99.06 0)
 			(hide yes)

Commit message: Footprint Assignment
Parts:
- SW2, SW3, SW4, SW5, SW6, SW7, SW8: footprint (none) -> Button_Switch_SMD:SW_SPST_B3U-1100P-B
Changed lines of the file:
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@@
 			)
 		)
-		(property "Footprint" ""
+		(property "Footprint" "Button_Switch_SMD:SW_SPST_B3U-1100P-B"
 			(at 191.77 105.41 0)
 			(hide yes)
@@
 			)
 		)
-		(property "Footprint" ""
+		(property "Footprint" "Button_Switch_SMD:SW_SPST_B3U-1100P-B"
 			(at 162.56 85.09 0)
 			(hide yes)
@@
 			)
 		)
-		(property "Footprint" ""
+		(property "Footprint" "Button_Switch_SMD:SW_SPST_B3U-1100P-B"
 			(at 220.98 85.09 0)
 			(hide yes)
@@
 			)
 		)
-		(property "Footprint" ""
+		(property "Footprint" "Button_Switch_SMD:SW_SPST_B3U-1100P-B"
 			(at 191.77 64.77 0)
 			(hide yes)
@@
 			)
 		)
-		(property "Footprint" ""
+		(property "Footprint" "Button_Switch_SMD:SW_SPST_B3U-1100P-B"
 			(at 60.96 67.31 0)
 			(hide yes)
@@
 			)
 		)
-		(property "Footprint" ""
+		(property "Footprint" "Button_Switch_SMD:SW_SPST_B3U-1100P-B"
 			(at 90.17 67.31 0)
 			(hide yes)
@@
 			)
 		)
-		(property "Footprint" ""
+		(property "Footprint" "Button_Switch_SMD:SW_SPST_B3U-1100P-B"
 			(at 191.77 85.09 0)
 			(hide yes)

Commit message: PCB Routing
Parts:
- SW2, SW3, SW4, SW5, SW6, SW7, SW8: footprint Button_Switch_SMD:SW_SPST_B3U-1100P-B -> (none); Mfr. Part # B3U-1100PM-B -> (none); Store URL - Digikey https://www.digikey.pt/pt/products/detail/aratas-formerly-o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 -> (none); Store URL - Mouser https://pt.mouser.com/en/ProductDetail/Omron-Electronics/B3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 -> (none)
Changed lines of the file:
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@@
 			)
 		)
-		(property "Footprint" "Button_Switch_SMD:SW_SPST_B3U-1100P-B"
+		(property "Footprint" ""
 			(at 191.77 105.41 0)
 			(hide yes)
@@
 			)
 		)
-		(property "Datasheet" "https://components.omron.com/us-en/sites/components.omron.com.us/files/datasheet_pdf/A162-E1.pdf"
+		(property "Datasheet" ""
 			(at 191.77 105.41 0)
 			(hide yes)
@@
 			)
 		)
-		(property "Description" "Push button switch, generic, two pins"
+		(property "Description" ""
 			(at 191.77 110.49 0)
 			(hide yes)
@@
 			)
 		)
-		(property "Mfr. Part #" "B3U-1100PM-B"
+		(property "Mfr. Part #" ""
 			(at 191.77 110.49 0)
 			(hide yes)
@@
 			)
 		)
-		(property "Store URL - Digikey" "https://www.digikey.pt/pt/products/detail/aratas-formerly-omron-components/B3U-1100PM-B/26811828?s=N4IgjCBcoGwJxVAYygMwIYBsDOBTANCAPZQDaIALAAxwDMdIAuoQA4AuUIAymwE4CWAOwDmIAL6EArACYAHIhApIGHAWJkQtWVVoxaTVh0jc%2BQ0RJCSYAdgVKVeQiUjlpVCrWm3mIdpx4CIuKEYHCyCNCKaFiO6i4gVExiyUA"
+		(property "Store URL - Digikey" ""
 			(at 191.77 110.49 0)
 			(hide yes)
@@
 			)
 		)
-		(property "Store URL - Mouser" "https://pt.mouser.com/en/ProductDetail/Omron-Electronics/B3U-1100PM-B?qs=hnUcNC2tU0rEzAhA%2F6P6YQ%3D%3D"
+		(property "Store URL - Mouser" ""
 			(at 191.77 110.49 0)
 			(hide yes)
@@
 			)
 		)
-		(property "Footprint" "Button_Switch_SMD:SW_SPST_B3U-1100P-B"
+		(property "Footprint" ""
 			(at 162.56 85.09 0)
 			(hide yes)
@@
 			)
 		)
-		(property "Datasheet" "https://components.omron.com/us-en/sites/components.omron.com.us/files/datasheet_pdf/A162-E1.pdf"
+		(property "Datasheet" ""
 			(at 162.56 85.09 0)
 			(hide yes)
@@
 			)
 		)
-		(property "Description" "Push button switch, generic, two pins"
+		(property "Description" ""
 			(at 162.56 90.17 0)
 			(hide yes)
@@
 			)
 		)
-		(property "Mfr. Part #" "B3U-1100PM-B"
+		(property "Mfr. Part #" ""
 			(at 162.56 90.17 0)
 			(hide yes)
@@
 			)
 		)
-		(property "Store URL - Digikey" "https://www.digikey.pt/pt/products/detail/aratas-formerly-omron-components/B3U-1100PM-B/26811828?s=N4IgjCBcoGwJxVAYygMwIYBsDOBTANCAPZQDaIALAAxwDMdIAuoQA4AuUIAymwE4CWAOwDmIAL6EArACYAHIhApIGHAWJkQtWVVoxaTVh0jc%2BQ0RJCSYAdgVKVeQiUjlpVCrWm3mIdpx4CIuKEYHCyCNCKaFiO6i4gVExiyUA"
+		(property "Store URL - Digikey" ""
 			(at 162.56 90.17 0)
 			(hide yes)
@@
 			)
 		)
-		(property "Store URL - Mouser" "https://pt.mouser.com/en/ProductDetail/Omron-Electronics/B3U-1100PM-B?qs=hnUcNC2tU0rEzAhA%2F6P6YQ%3D%3D"
+		(property "Store URL - Mouser" ""
 			(at 162.56 90.17 0)
 			(hide yes)
@@
 			)
 		)
-		(property "Footprint" "Button_Switch_SMD:SW_SPST_B3U-1100P-B"
+		(property "Footprint" ""
 			(at 220.98 85.09 0)
 			(hide yes)
@@
 			)
 		)
-		(property "Datasheet" "https://components.omron.com/us-en/sites/components.omron.com.us/files/datasheet_pdf/A162-E1.pdf"
+		(property "Datasheet" ""
 			(at 220.98 85.09 0)
 			(hide yes)
@@
 			)
 		)
-		(property "Description" "Push button switch, generic, two pins"
+		(property "Description" ""
 			(at 220.98 90.17 0)
 			(hide yes)
@@
 			)
 		)
-		(property "Mfr. Part #" "B3U-1100PM-B"
+		(property "Mfr. Part #" ""
 			(at 220.98 90.17 0)
 			(hide yes)
@@
 			)
 		)
-		(property "Store URL - Digikey" "https://www.digikey.pt/pt/products/detail/aratas-formerly-omron-components/B3U-1100PM-B/26811828?s=N4IgjCBcoGwJxVAYygMwIYBsDOBTANCAPZQDaIALAAxwDMdIAuoQA4AuUIAymwE4CWAOwDmIAL6EArACYAHIhApIGHAWJkQtWVVoxaTVh0jc%2BQ0RJCSYAdgVKVeQiUjlpVCrWm3mIdpx4CIuKEYHCyCNCKaFiO6i4gVExiyUA"
+		(property "Store URL - Digikey" ""
 			(at 220.98 90.17 0)
 			(hide yes)
@@
 			)
 		)
-		(property "Store URL - Mouser" "https://pt.mouser.com/en/ProductDetail/Omron-Electronics/B3U-1100PM-B?qs=hnUcNC2tU0rEzAhA%2F6P6YQ%3D%3D"
+		(property "Store URL - Mouser" ""
 			(at 220.98 90.17 0)
 			(hide yes)
@@
 			)
 		)
-		(property "Footprint" "Button_Switch_SMD:SW_SPST_B3U-1100P-B"
+		(property "Footprint" ""
 			(at 191.77 64.77 0)
 			(hide yes)
@@
 			)
 		)
-		(property "Datasheet" "https://components.omron.com/us-en/sites/components.omron.com.us/files/datasheet_pdf/A162-E1.pdf"
+		(property "Datasheet" ""
 			(at 191.77 64.77 0)
 			(hide yes)
@@
 			)
 		)
-		(property "Description" "Push button switch, generic, two pins"
+		(property "Description" ""
 			(at 191.77 69.85 0)
 			(hide yes)
@@
 			)
 		)
-		(property "Mfr. Part #" "B3U-1100PM-B"
+		(property "Mfr. Part #" ""
 			(at 191.77 69.85 0)
 			(hide yes)
@@
 			)
 		)
-		(property "Store URL - Digikey" "https://www.digikey.pt/pt/products/detail/aratas-formerly-omron-components/B3U-1100PM-B/26811828?s=N4IgjCBcoGwJxVAYygMwIYBsDOBTANCAPZQDaIALAAxwDMdIAuoQA4AuUIAymwE4CWAOwDmIAL6EArACYAHIhApIGHAWJkQtWVVoxaTVh0jc%2BQ0RJCSYAdgVKVeQiUjlpVCrWm3mIdpx4CIuKEYHCyCNCKaFiO6i4gVExiyUA"
+		(property "Store URL - Digikey" ""
 			(at 191.77 69.85 0)
 			(hide yes)
@@
 			)
 		)
-		(property "Store URL - Mouser" "https://pt.mouser.com/en/ProductDetail/Omron-Electronics/B3U-1100PM-B?qs=hnUcNC2tU0rEzAhA%2F6P6YQ%3D%3D"
+		(property "Store URL - Mouser" ""
 			(at 191.77 69.85 0)
 			(hide yes)
@@
 			)
 		)
-		(property "Footprint" "Button_Switch_SMD:SW_SPST_B3U-1100P-B"
+		(property "Footprint" ""
 			(at 60.96 67.31 0)
 			(hide yes)
@@
 			)
 		)
-		(property "Datasheet" "https://components.omron.com/us-en/sites/components.omron.com.us/files/datasheet_pdf/A162-E1.pdf"
+		(property "Datasheet" ""
 			(at 60.96 67.31 0)
 			(hide yes)
@@
 			)
 		)
-		(property "Description" "Push button switch, generic, two pins"
+		(property "Description" ""
 			(at 60.96 72.39 0)
 			(hide yes)
@@
 			)
 		)
-		(property "Mfr. Part #" "B3U-1100PM-B"
+		(property "Mfr. Part #" ""
 			(at 60.96 72.39 0)
 			(hide yes)
@@
 			)
 		)
-		(property "Store URL - Digikey" "https://www.digikey.pt/pt/products/detail/aratas-formerly-omron-components/B3U-1100PM-B/26811828?s=N4IgjCBcoGwJxVAYygMwIYBsDOBTANCAPZQDaIALAAxwDMdIAuoQA4AuUIAymwE4CWAOwDmIAL6EArACYAHIhApIGHAWJkQtWVVoxaTVh0jc%2BQ0RJCSYAdgVKVeQiUjlpVCrWm3mIdpx4CIuKEYHCyCNCKaFiO6i4gVExiyUA"
+		(property "Store URL - Digikey" ""
 			(at 60.96 72.39 0)
 			(hide yes)
@@
 			)
 		)
-		(property "Store URL - Mouser" "https://pt.mouser.com/en/ProductDetail/Omron-Electronics/B3U-1100PM-B?qs=hnUcNC2tU0rEzAhA%2F6P6YQ%3D%3D"
+		(property "Store URL - Mouser" ""
 			(at 60.96 72.39 0)
 			(hide yes)
@@
 			)
 		)
-		(property "Footprint" "Button_Switch_SMD:SW_SPST_B3U-1100P-B"
+		(property "Footprint" ""
 			(at 90.17 67.31 0)
 			(hide yes)
@@
 			)
 		)
-		(property "Datasheet" "https://components.omron.com/us-en/sites/components.omron.com.us/files/datasheet_pdf/A162-E1.pdf"
+		(property "Datasheet" ""
 			(at 90.17 67.31 0)
 			(hide yes)
@@
 			)
 		)
-		(property "Description" "Push button switch, generic, two pins"
+		(property "Description" ""
 			(at 90.17 72.39 0)
 			(hide yes)
@@
 			)
 		)
-		(property "Mfr. Part #" "B3U-1100PM-B"
+		(property "Mfr. Part #" ""
 			(at 90.17 72.39 0)
 			(hide yes)
@@
 			)
 		)
-		(property "Store URL - Digikey" "https://www.digikey.pt/pt/products/detail/aratas-formerly-omron-components/B3U-1100PM-B/26811828?s=N4IgjCBcoGwJxVAYygMwIYBsDOBTANCAPZQDaIALAAxwDMdIAuoQA4AuUIAymwE4CWAOwDmIAL6EArACYAHIhApIGHAWJkQtWVVoxaTVh0jc%2BQ0RJCSYAdgVKVeQiUjlpVCrWm3mIdpx4CIuKEYHCyCNCKaFiO6i4gVExiyUA"
+		(property "Store URL - Digikey" ""
 			(at 90.17 72.39 0)
 			(hide yes)
@@
 			)
 		)
-		(property "Store URL - Mouser" "https://pt.mouser.com/en/ProductDetail/Omron-Electronics/B3U-1100PM-B?qs=hnUcNC2tU0rEzAhA%2F6P6YQ%3D%3D"
+		(property "Store URL - Mouser" ""
 			(at 90.17 72.39 0)
 			(hide yes)
@@
 			)
 		)
-		(property "Footprint" "Button_Switch_SMD:SW_SPST_B3U-1100P-B"
+		(property "Footprint" ""
 			(at 191.77 85.09 0)
 			(hide yes)
@@
 			)
 		)
-		(property "Datasheet" "https://components.omron.com/us-en/sites/components.omron.com.us/files/datasheet_pdf/A162-E1.pdf"
+		(property "Datasheet" ""
 			(at 191.77 85.09 0)
 			(hide yes)
@@
 			)
 		)
-		(property "Description" "Push button switch, generic, two pins"
+		(property "Description" ""
 			(at 191.77 90.17 0)
 			(hide yes)
@@
 			)
 		)
-		(property "Mfr. Part #" "B3U-1100PM-B"
+		(property "Mfr. Part #" ""
 			(at 191.77 90.17 0)
 			(hide yes)
@@
 			)
 		)
-		(property "Store URL - Digikey" "https://www.digikey.pt/pt/products/detail/aratas-formerly-omron-components/B3U-1100PM-B/26811828?s=N4IgjCBcoGwJxVAYygMwIYBsDOBTANCAPZQDaIALAAxwDMdIAuoQA4AuUIAymwE4CWAOwDmIAL6EArACYAHIhApIGHAWJkQtWVVoxaTVh0jc%2BQ0RJCSYAdgVKVeQiUjlpVCrWm3mIdpx4CIuKEYHCyCNCKaFiO6i4gVExiyUA"
+		(property "Store URL - Digikey" ""
 			(at 191.77 90.17 0)
 			(hide yes)
@@
 			)
 		)
-		(property "Store URL - Mouser" "https://pt.mouser.com/en/ProductDetail/Omron-Electronics/B3U-1100PM-B?qs=hnUcNC2tU0rEzAhA%2F6P6YQ%3D%3D"
+		(property "Store URL - Mouser" ""
 			(at 191.77 90.17 0)
 			(hide yes)

Commit message: PCB Routing
Parts:
- SW2, SW3, SW4, SW5, SW6, SW7, SW8: footprint (none) -> Button_Switch_SMD:SW_Push_SPST_NO_Alps_SKRK; Mfr. Part # (none) -> TL1017ABAF260QG; Store URL - Digikey (none) -> https://www.digikey.pt/pt/products/detail/e-switch/TL1017AB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; Store URL - Mouser (none) -> https://eu.mouser.com/en/ProductDetail/E-Switch/TL1017ABAF2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
Changed lines of the file:
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@@
 			)
 		)
-		(property "Footprint" ""
+		(property "Footprint" "Button_Switch_SMD:SW_Push_SPST_NO_Alps_SKRK"
 			(at 191.77 105.41 0)
 			(hide yes)
@@
 			)
 		)
-		(property "Datasheet" ""
+		(property "Datasheet" "https://configured-product-images.s3.amazonaws.com/Datasheets/TL1017.pdf"
 			(at 191.77 105.41 0)
 			(hide yes)
@@
 			)
 		)
-		(property "Description" ""
+		(property "Description" "Interruptor tátil SPST-NA Top atuado Montagem em superfície"
 			(at 191.77 110.49 0)
 			(hide yes)
@@
 			)
 		)
-		(property "Mfr. Part #" ""
+		(property "Mfr. Part #" "TL1017ABAF260QG"
 			(at 191.77 110.49 0)
 			(hide yes)
@@
 			)
 		)
-		(property "Store URL - Digikey" ""
+		(property "Store URL - Digikey" "https://www.digikey.pt/pt/products/detail/e-switch/TL1017ABAF260QG/18687016"
 			(at 191.77 110.49 0)
 			(hide yes)
@@
 			)
 		)
-		(property "Store URL - Mouser" ""
+		(property "Store URL - Mouser" "https://eu.mouser.com/en/ProductDetail/E-Switch/TL1017ABAF260QG?qs=9vOqFld9vZVWa2gSWDc0aQ%3D%3D"
 			(at 191.77 110.49 0)
 			(hide yes)
@@
 			)
 		)
-		(property "Footprint" ""
+		(property "Footprint" "Button_Switch_SMD:SW_Push_SPST_NO_Alps_SKRK"
 			(at 162.56 85.09 0)
 			(hide yes)
@@
 			)
 		)
-		(property "Datasheet" ""
+		(property "Datasheet" "https://configured-product-images.s3.amazonaws.com/Datasheets/TL1017.pdf"
 			(at 162.56 85.09 0)
 			(hide yes)
@@
 			)
 		)
-		(property "Description" ""
+		(property "Description" "Interruptor tátil SPST-NA Top atuado Montagem em superfície"
 			(at 162.56 90.17 0)
 			(hide yes)
@@
 			)
 		)
-		(property "Mfr. Part #" ""
+		(property "Mfr. Part #" "TL1017ABAF260QG"
 			(at 162.56 90.17 0)
 			(hide yes)
@@
 			)
 		)
-		(property "Store URL - Digikey" ""
+		(property "Store URL - Digikey" "https://www.digikey.pt/pt/products/detail/e-switch/TL1017ABAF260QG/18687016"
 			(at 162.56 90.17 0)
 			(hide yes)
@@
 			)
 		)
-		(property "Store URL - Mouser" ""
+		(property "Store URL - Mouser" "https://eu.mouser.com/en/ProductDetail/E-Switch/TL1017ABAF260QG?qs=9vOqFld9vZVWa2gSWDc0aQ%3D%3D"
 			(at 162.56 90.17 0)
 			(hide yes)
@@
 			)
 		)
-		(property "Footprint" ""
+		(property "Footprint" "Button_Switch_SMD:SW_Push_SPST_NO_Alps_SKRK"
 			(at 220.98 85.09 0)
 			(hide yes)
@@
 			)
 		)
-		(property "Datasheet" ""
+		(property "Datasheet" "https://configured-product-images.s3.amazonaws.com/Datasheets/TL1017.pdf"
 			(at 220.98 85.09 0)
 			(hide yes)
@@
 			)
 		)
-		(property "Description" ""
+		(property "Description" "Interruptor tátil SPST-NA Top atuado Montagem em superfície"
 			(at 220.98 90.17 0)
 			(hide yes)
@@
 			)
 		)
-		(property "Mfr. Part #" ""
+		(property "Mfr. Part #" "TL1017ABAF260QG"
 			(at 220.98 90.17 0)
 			(hide yes)
@@
 			)
 		)
-		(property "Store URL - Digikey" ""
+		(property "Store URL - Digikey" "https://www.digikey.pt/pt/products/detail/e-switch/TL1017ABAF260QG/18687016"
 			(at 220.98 90.17 0)
 			(hide yes)
@@
 			)
 		)
-		(property "Store URL - Mouser" ""
+		(property "Store URL - Mouser" "https://eu.mouser.com/en/ProductDetail/E-Switch/TL1017ABAF260QG?qs=9vOqFld9vZVWa2gSWDc0aQ%3D%3D"
 			(at 220.98 90.17 0)
 			(hide yes)
@@
 			)
 		)
-		(property "Footprint" ""
+		(property "Footprint" "Button_Switch_SMD:SW_Push_SPST_NO_Alps_SKRK"
 			(at 191.77 64.77 0)
 			(hide yes)
@@
 			)
 		)
-		(property "Datasheet" ""
+		(property "Datasheet" "https://configured-product-images.s3.amazonaws.com/Datasheets/TL1017.pdf"
 			(at 191.77 64.77 0)
 			(hide yes)
@@
 			)
 		)
-		(property "Description" ""
+		(property "Description" "Interruptor tátil SPST-NA Top atuado Montagem em superfície"
 			(at 191.77 69.85 0)
 			(hide yes)
@@
 			)
 		)
-		(property "Mfr. Part #" ""
+		(property "Mfr. Part #" "TL1017ABAF260QG"
 			(at 191.77 69.85 0)
 			(hide yes)
@@
 			)
 		)
-		(property "Store URL - Digikey" ""
+		(property "Store URL - Digikey" "https://www.digikey.pt/pt/products/detail/e-switch/TL1017ABAF260QG/18687016"
 			(at 191.77 69.85 0)
 			(hide yes)
@@
 			)
 		)
-		(property "Store URL - Mouser" ""
+		(property "Store URL - Mouser" "https://eu.mouser.com/en/ProductDetail/E-Switch/TL1017ABAF260QG?qs=9vOqFld9vZVWa2gSWDc0aQ%3D%3D"
 			(at 191.77 69.85 0)
 			(hide yes)
@@
 			)
 		)
-		(property "Footprint" ""
+		(property "Footprint" "Button_Switch_SMD:SW_Push_SPST_NO_Alps_SKRK"
 			(at 60.96 67.31 0)
 			(hide yes)
@@
 			)
 		)
-		(property "Datasheet" ""
+		(property "Datasheet" "https://configured-product-images.s3.amazonaws.com/Datasheets/TL1017.pdf"
 			(at 60.96 67.31 0)
 			(hide yes)
@@
 			)
 		)
-		(property "Description" ""
+		(property "Description" "Interruptor tátil SPST-NA Top atuado Montagem em superfície"
 			(at 60.96 72.39 0)
 			(hide yes)
@@
 			)
 		)
-		(property "Mfr. Part #" ""
+		(property "Mfr. Part #" "TL1017ABAF260QG"
 			(at 60.96 72.39 0)
 			(hide yes)
@@
 			)
 		)
-		(property "Store URL - Digikey" ""
+		(property "Store URL - Digikey" "https://www.digikey.pt/pt/products/detail/e-switch/TL1017ABAF260QG/18687016"
 			(at 60.96 72.39 0)
 			(hide yes)
@@
 			)
 		)
-		(property "Store URL - Mouser" ""
+		(property "Store URL - Mouser" "https://eu.mouser.com/en/ProductDetail/E-Switch/TL1017ABAF260QG?qs=9vOqFld9vZVWa2gSWDc0aQ%3D%3D"
 			(at 60.96 72.39 0)
 			(hide yes)
@@
 			)
 		)
-		(property "Footprint" ""
+		(property "Footprint" "Button_Switch_SMD:SW_Push_SPST_NO_Alps_SKRK"
 			(at 90.17 67.31 0)
 			(hide yes)
@@
 			)
 		)
-		(property "Datasheet" ""
+		(property "Datasheet" "https://configured-product-images.s3.amazonaws.com/Datasheets/TL1017.pdf"
 			(at 90.17 67.31 0)
 			(hide yes)
@@
 			)
 		)
-		(property "Description" ""
+		(property "Description" "Interruptor tátil SPST-NA Top atuado Montagem em superfície"
 			(at 90.17 72.39 0)
 			(hide yes)
@@
 			)
 		)
-		(property "Mfr. Part #" ""
+		(property "Mfr. Part #" "TL1017ABAF260QG"
 			(at 90.17 72.39 0)
 			(hide yes)
@@
 			)
 		)
-		(property "Store URL - Digikey" ""
+		(property "Store URL - Digikey" "https://www.digikey.pt/pt/products/detail/e-switch/TL1017ABAF260QG/18687016"
 			(at 90.17 72.39 0)
 			(hide yes)
@@
 			)
 		)
-		(property "Store URL - Mouser" ""
+		(property "Store URL - Mouser" "https://eu.mouser.com/en/ProductDetail/E-Switch/TL1017ABAF260QG?qs=9vOqFld9vZVWa2gSWDc0aQ%3D%3D"
 			(at 90.17 72.39 0)
 			(hide yes)
@@
 			)
 		)
-		(property "Footprint" ""
+		(property "Footprint" "Button_Switch_SMD:SW_Push_SPST_NO_Alps_SKRK"
 			(at 191.77 85.09 0)
 			(hide yes)
@@
 			)
 		)
-		(property "Datasheet" ""
+		(property "Datasheet" "https://configured-product-images.s3.amazonaws.com/Datasheets/TL1017.pdf"
 			(at 191.77 85.09 0)
 			(hide yes)
@@
 			)
 		)
-		(property "Description" ""
+		(property "Description" "Interruptor tátil SPST-NA Top atuado Montagem em superfície"
 			(at 191.77 90.17 0)
 			(hide yes)
@@
 			)
 		)
-		(property "Mfr. Part #" ""
+		(property "Mfr. Part #" "TL1017ABAF260QG"
 			(at 191.77 90.17 0)
 			(hide yes)
@@
 			)
 		)
-		(property "Store URL - Digikey" ""
+		(property "Store URL - Digikey" "https://www.digikey.pt/pt/products/detail/e-switch/TL1017ABAF260QG/18687016"
 			(at 191.77 90.17 0)
 			(hide yes)
@@
 			)
 		)
-		(property "Store URL - Mouser" ""
+		(property "Store URL - Mouser" "https://eu.mouser.com/en/ProductDetail/E-Switch/TL1017ABAF260QG?qs=9vOqFld9vZVWa2gSWDc0aQ%3D%3D"
 			(at 191.77 90.17 0)
 			(hide yes)
