File: PCB/MP3_Player/power.kicad_sch (KiCad schematic)
At the start: 18 parts, among them J5 BAT Connector, SW1 Toggle Switch, U2 AP2112K-3.3, U3 BQ24075RGTR, U5 MAX17048G

Commit message: Final PCB Routing
Connections:
- net TS: now reaches R9.1, U3.1 (TS)
Changed lines of the file:
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@@
+		)
+	)
+	(label "TS"
+		(at 115.57 91.44 0)
+		(effects
+			(font
+				(size 1.27 1.27)
+			)
+			(justify left bottom)
 		)
 	)
@@
 		(effects
 			(font
+				(size 1.27 1.27)
+			)
+			(justify left bottom)
+		)
+	)
+	(label "EN1"
+		(at 86.36 69.85 0)
+		(effects
+			(font
