File: PCB/MP3_Player/wireless.kicad_sch (KiCad schematic)
At the start: 14 parts, among them U7 ST67W611M1A6B, Y3 32.768KHz

Commit message: Minor Schematic Changes
Other:
- note added: "Bridge when programming"
- moved on the sheet: C34, JP1, R16, R25

Commit message: Started Making BOM
Parts:
- C28: Mfr. Part # (none) -> CL10A106KP8NNNC; Store URL - Digikey (none) -> https://www.digikey.pt/pt/products/detail/samsung-electro-m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; Store URL - Mouser (none) -> https://pt.mouser.com/en/ProductDetail/Samsung-Electro-Mech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
- C29, C30, C31, C34: Mfr. Part # (none) -> CL05B104KP5NNNC; Store URL - Digikey (none) -> https://www.digikey.pt/pt/products/detail/samsung-electro-m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; Store URL - Mouser (none) -> https://pt.mouser.com/en/ProductDetail/Samsung-Electro-Mech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
- C32, C33: Mfr. Part # (none) -> CL05C2R2CB51PNC; Store URL - Digikey (none) -> https://www.digikey.pt/pt/products/detail/samsung-electro-m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; Store URL - Mouser (none) -> https://pt.mouser.com/en/ProductDetail/Samsung-Electro-Mech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
- TP1, TP2: now left out of the parts list

Commit message: Continue Making BOM
Parts:
- R16, R25: Mfr. Part # (none) -> CRCW040210K0FKED; Store URL - Digikey (none) -> https://www.digikey.pt/pt/products/detail/vishay-dale/CRCW0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; Store URL - Mouser (none) -> https://pt.mouser.com/en/ProductDetail/Vishay/CRCW040210K0F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
Changed lines of the file:
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@@
 			)
 		)
-		(property "Datasheet" ""
+		(property "Datasheet" "https://www.vishay.com/docs/20035/dcrcwe3.pdf"
 			(at 179.07 74.93 0)
 			(hide yes)
@@
 			)
 		)
-		(property "Description" "Resistor"
+		(property "Description" "0402"
 			(at 179.07 74.93 0)
 			(hide yes)
@@
 		)
 		(property "Store URL - TME" ""
+			(at 179.07 74.93 0)
+			(hide yes)
+			(show_name no)
+			(do_not_autoplace no)
+			(effects
+				(font
+					(size 1.27 1.27)
+				)
+			)
+		)
+		(property "Mfr. Part #" "CRCW040210K0FKED"
+			(at 179.07 74.93 0)
+			(hide yes)
+			(show_name no)
+			(do_not_autoplace no)
+			(effects
+				(font
+					(size 1.27 1.27)
+				)
+			)
+		)
+		(property "Store URL - Digikey" "https://www.digikey.pt/pt/products/detail/vishay-dale/CRCW040210K0FKED/1178121"
+			(at 179.07 74.93 0)
+			(hide yes)
+			(show_name no)
+			(do_not_autoplace no)
+			(effects
+				(font
+					(size 1.27 1.27)
+				)
+			)
+		)
+		(property "Store URL - Mouser" "https://pt.mouser.com/en/ProductDetail/Vishay/CRCW040210K0FKED?qs=rlE3Te1NifyN3e8vvxacSw%3D%3D"
 			(at 179.07 74.93 0)
 			(hide yes)
@@
 			)
 		)
-		(property "Datasheet" ""
+		(property "Datasheet" "https://www.vishay.com/docs/20035/dcrcwe3.pdf"
 			(at 162.56 69.85 0)
 			(hide yes)
@@
 			)
 		)
-		(property "Description" "Resistor"
+		(property "Description" "0402"
 			(at 162.56 69.85 0)
 			(hide yes)
@@
 			(at 162.56 69.85 90)
 			(hide yes)
+			(show_name no)
+			(do_not_autoplace no)
+			(effects
+				(font
+					(size 1.27 1.27)
+				)
+			)
+		)
+		(property "Mfr. Part #" "CRCW040210K0FKED"
+			(at 162.56 69.85 90)
+			(hide yes)
+			(show_name no)
+			(do_not_autoplace no)
+			(effects
+				(font
+					(size 1.27 1.27)
+				)
+			)
+		)
+		(property "Store URL - Digikey" "https://www.digikey.pt/pt/products/detail/vishay-dale/CRCW040210K0FKED/1178121"
+			(at 162.56 69.85 90)
+			(hide yes)
+			(show_name no)
+			(do_not_autoplace no)
+			(effects
+				(font
+					(size 1.27 1.27)
+				)
+			)
+		)
+		(property "Store URL - Mouser" "https://pt.mouser.com/en/ProductDetail/Vishay/CRCW040210K0FKED?qs=rlE3Te1NifyN3e8vvxacSw%3D%3D"
+			(at 162.56 69.85 90)
+			(hide yes)

Commit message: Finished BOM; Started Footprint assignment
Parts:
- C28: footprint (none) -> Capacitor_SMD:C_0603_1608Metric
- C29, C30, C31, C32, C33, C34, R16, R25: footprint (none) -> Capacitor_SMD:C_0402_1005Metric
Changed lines of the file:
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@@
 			)
 		)
-		(property "Footprint" ""
+		(property "Footprint" "Capacitor_SMD:C_0402_1005Metric"
 			(at 177.292 74.93 90)
 			(hide yes)
@@
 			)
 		)
-		(property "Footprint" ""
+		(property "Footprint" "Capacitor_SMD:C_0402_1005Metric"
 			(at 182.5752 106.68 0)
 			(hide yes)
@@
 			)
 		)
-		(property "Footprint" ""
+		(property "Footprint" "Capacitor_SMD:C_0402_1005Metric"
 			(at 96.2152 54.61 0)
 			(hide yes)
@@
 			)
 		)
-		(property "Footprint" ""
+		(property "Footprint" "Capacitor_SMD:C_0603_1608Metric"
 			(at 84.7852 54.61 0)
 			(hide yes)
@@
 			)
 		)
-		(property "Footprint" ""
+		(property "Footprint" "Capacitor_SMD:C_0402_1005Metric"
 			(at 162.56 71.628 90)
 			(hide yes)
@@
 			)
 		)
-		(property "Footprint" ""
+		(property "Footprint" "Capacitor_SMD:C_0402_1005Metric"
 			(at 107.6452 54.61 0)
 			(hide yes)
@@
 			)
 		)
-		(property "Footprint" ""
+		(property "Footprint" "Capacitor_SMD:C_0402_1005Metric"
 			(at 158.75 63.8048 0)
 			(hide yes)
@@
 			)
 		)
-		(property "Footprint" ""
+		(property "Footprint" "Capacitor_SMD:C_0402_1005Metric"
 			(at 119.0752 54.61 0)
 			(hide yes)
@@
 			)
 		)
-		(property "Footprint" ""
+		(property "Footprint" "Capacitor_SMD:C_0402_1005Metric"
 			(at 167.9448 106.68 0)
 			(hide yes)

Commit message: Footprint Assingment
Parts:
- JP1: footprint (none) -> Jumper:SolderJumper-2_P1.3mm_Bridged2Bar_RoundedPad1.0x1.5mm
- R16, R25: footprint Capacitor_SMD:C_0402_1005Metric -> Resistor_SMD:R_0402_1005Metric
- TP1, TP2: footprint Relay_THT:Relay_DPDT_Schrack-RT2-FormC_RM5mm -> TestPoint:TestPoint_Pad_D1.5mm
Changed lines of the file:
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@@
 			)
 		)
-		(property "Footprint" "Capacitor_SMD:C_0402_1005Metric"
+		(property "Footprint" "Resistor_SMD:R_0402_1005Metric"
 			(at 177.292 74.93 90)
 			(hide yes)
@@
 			)
 		)
-		(property "Footprint" "Relay_THT:Relay_DPDT_Schrack-RT2-FormC_RM5mm"
+		(property "Footprint" "TestPoint:TestPoint_Pad_D1.5mm"
 			(at 110.49 68.58 0)
 			(hide yes)
@@
 			)
 		)
-		(property "Footprint" "Relay_THT:Relay_DPDT_Schrack-RT2-FormC_RM5mm"
+		(property "Footprint" "TestPoint:TestPoint_Pad_D1.5mm"
 			(at 110.49 81.28 0)
 			(hide yes)
@@
 			)
 		)
-		(property "Footprint" ""
+		(property "Footprint" "Jumper:SolderJumper-2_P1.3mm_Bridged2Bar_RoundedPad1.0x1.5mm"
 			(at 186.69 69.85 0)
 			(hide yes)
@@
 			)
 		)
-		(property "Footprint" "Capacitor_SMD:C_0402_1005Metric"
+		(property "Footprint" "Resistor_SMD:R_0402_1005Metric"
 			(at 162.56 71.628 90)
 			(hide yes)

Commit message: Footprint Assingment Complete
Parts:
- TP1, TP2: footprint TestPoint:TestPoint_Pad_D1.5mm -> TestPoint:TestPoint_Pad_D1.0mm
Changed lines of the file:
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@@
 			)
 		)
-		(property "Footprint" "TestPoint:TestPoint_Pad_D1.5mm"
+		(property "Footprint" "TestPoint:TestPoint_Pad_D1.0mm"
 			(at 110.49 68.58 0)
 			(hide yes)
@@
 			)
 		)
-		(property "Footprint" "TestPoint:TestPoint_Pad_D1.5mm"
+		(property "Footprint" "TestPoint:TestPoint_Pad_D1.0mm"
 			(at 110.49 81.28 0)
 			(hide yes)

Commit message: PCB Layout
Connections:
- net Boot Select: now reaches JP1.1 (A), R25.1, U7.3 (BOOT)
Changed lines of the file:
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@@
+		)
+	)
+	(label "Boot Select"
+		(at 158.75 77.47 0)
+		(effects
+			(font
+				(size 1.27 1.27)
+			)
+			(justify left bottom)
 		)
 	)

Commit message: Final PCB Routing
Connections:
- net XTAL_OUT: now reaches C33.1, U7.13 (XTAL32K_OUT), Y3.2
- net XATL_IN: now reaches C32.1, U7.14 (XTAL32K_IN), Y3.1
- net UART_TX: now reaches TP1.1, U7.22 (UART_TX)
- net UART_RX: now reaches TP2.1, U7.23 (UART_RX)
Other:
- moved on the sheet: TP1, TP2
Changed lines of the file:
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@@
+	(wire
+		(pts
+			(xy 102.87 73.66) (xy 110.49 73.66)
+		)
+		(stroke
+			(width 0)
+			(type default)
+		)
+	)
 	(wire
 		(pts
@@
 	(wire
 		(pts
+			(xy 102.87 76.2) (xy 110.49 76.2)
+		)
+		(stroke
+			(width 0)
+			(type default)
+		)
+	)
+	(wire
+		(pts
 			(xy 158.75 64.77) (xy 157.48 64.77)
 		)
@@
 			(width 0)
 			(type default)
+		)
+	)
+	(label "XATL_IN"
+		(at 157.48 86.36 0)
+		(effects
+			(font
+				(size 1.27 1.27)
+			)
+			(justify left bottom)
+		)
+	)
+	(label "XTAL_OUT"
+		(at 157.48 88.9 0)
+		(effects
+			(font
+				(size 1.27 1.27)
+			)
+			(justify left bottom)
 		)
 	)
@@
 		(effects
 			(font
-				(size 1.27 1.27)
+				(size 0.635 0.635)
+			)
+			(justify left bottom)
+		)
+	)
+	(label "UART_TX"
+		(at 104.14 73.66 0)
+		(effects
+			(font
+				(size 0.635 0.635)
+			)
+			(justify left bottom)
+		)
+	)
+	(label "UART_RX"
+		(at 104.0984 76.2 0)
+		(effects
+			(font
+				(size 0.635 0.635)
 			)
 			(justify left bottom)
@@
 	(symbol
 		(lib_id "Connector:TestPoint")
-		(at 110.49 73.66 90)
+		(at 102.87 73.66 90)
 		(unit 1)
 		(body_style 1)
@@
 		(fields_autoplaced yes)
 		(property "Reference" "TP1"
-			(at 107.188 68.58 90)
+			(at 99.568 68.58 90)
 			(show_name no)
 			(do_not_autoplace no)
@@
 		)
 		(property "Value" "UART_TX"
-			(at 107.188 71.12 90)
+			(at 99.568 71.12 90)
 			(show_name no)
 			(do_not_autoplace no)
@@
 		)
 		(property "Footprint" "TestPoint:TestPoint_Pad_D1.0mm"
-			(at 110.49 68.58 0)
+			(at 102.87 68.58 0)
 			(hide yes)
 			(show_name no)
@@
 		)
 		(property "Datasheet" ""
-			(at 110.49 68.58 0)
+			(at 102.87 68.58 0)
 			(hide yes)
 			(show_name no)
@@
 		)
 		(property "Description" "test point"
-			(at 110.49 73.66 0)
+			(at 102.87 73.66 0)
 			(hide yes)
 			(show_name no)
@@
 		)
 		(property "Store URL - Other" ""
-			(at 110.49 73.66 90)
+			(at 102.87 73.66 90)
 			(hide yes)
 			(show_name no)
@@
 		)
 		(property "Store URL - TME" ""
-			(at 110.49 73.66 90)
+			(at 102.87 73.66 90)
 			(hide yes)
 			(show_name no)
@@
 	(symbol
 		(lib_id "Connector:TestPoint")
-		(at 110.49 76.2 90)
+		(at 102.87 76.2 90)
 		(mirror x)
 		(unit 1)
@@
 		(dnp no)
 		(property "Reference" "TP2"
-			(at 107.188 81.28 90)
+			(at 99.568 81.28 90)
 			(show_name no)
 			(do_not_autoplace no)
@@
 		)
 		(property "Value" "UART_RX"
-			(at 107.188 78.74 90)
+			(at 99.568 78.74 90)
 			(show_name no)
 			(do_not_autoplace no)
@@
 		)
 		(property "Footprint" "TestPoint:TestPoint_Pad_D1.0mm"
-			(at 110.49 81.28 0)
+			(at 102.87 81.28 0)
 			(hide yes)
 			(show_name no)
@@
 		)
 		(property "Datasheet" ""
-			(at 110.49 81.28 0)
+			(at 102.87 81.28 0)
 			(hide yes)
 			(show_name no)
@@
 		)
 		(property "Description" "test point"
-			(at 110.49 76.2 0)
+			(at 102.87 76.2 0)
 			(hide yes)
 			(show_name no)
@@
 		)
 		(property "Store URL - Other" ""
-			(at 110.49 76.2 90)
+			(at 102.87 76.2 90)
 			(hide yes)
 			(show_name no)
@@
 		)
 		(property "Store URL - TME" ""
-			(at 110.49 76.2 90)
-			(hide yes)
-			(show_name no)
+			(at 102.87 76.2 90)
+			(hide yes)
+			(show_name no)
