File: PCB/MP3_Player/display.kicad_sch (KiCad schematic)
At the start: 8 parts, among them Q1 S8050

Commit message: PCB Correction
Parts:
- FCON1: footprint Connector_FFC-FPC:Amphenol_F32R-1A7x1-11025_1x25-1MP_P0.5mm_Horizontal -> Connector_FFC-FPC:Amphenol_F32R-1A7x1-11026_1x26-1MP_P0.5mm_Horizontal
Changed lines of the file:
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@@
 			)
 		)
-		(property "Footprint" "Connector_FFC-FPC:Amphenol_F32R-1A7x1-11025_1x25-1MP_P0.5mm_Horizontal"
+		(property "Footprint" "Connector_FFC-FPC:Amphenol_F32R-1A7x1-11026_1x26-1MP_P0.5mm_Horizontal"
 			(at 176.53 100.33 0)
 			(hide yes)
